File: eagle/max10adc dpdt.brd (EAGLE design)
At the start: 98 x 62 mm, 205 parts, among them IC1 MAX19506, IC2 MAX19506, J1 MOLEX_BNC_73100-0105, J2 MOLEX_BNC_73100-0105, J3 MOLEX_BNC_73100-0105, J4 MOLEX_BNC_73100-0105, K1 AQY21SOP, K2 AQY21SOP, K3 AQY21SOP, K4 AQY21SOP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

Commit message: dpdt
Parts:
- moved ST4 183.7 mm to (71.2, 57.3)
- moved ST3 149.5 mm to (71.4, 34.0)
- moved SSUPER4 136.2 mm to (60.3, 57.3), turned to 180 degrees
- moved ST2 128.7 mm to (71.5, 24.4)
- moved SSUPER3 104.8 mm to (61.0, 34.0), turned to 180 degrees
- moved SSUPER2 87.5 mm to (61.1, 24.4), turned to 180 degrees
- moved SSUPER1 41.3 mm to (60.3, 0.70), turned to 180 degrees
- moved ST1 39.3 mm to (71.2, 0.70)
- moved RIN4 0.60 mm to (71.0, 47.6)
- moved CL3 0.58 mm to (66.1, 39.2)
- moved CH3 0.50 mm to (70.1, 39.2)
- moved CH4 0.50 mm to (69.6, 52.0)
- moved CL4 0.50 mm to (65.9, 52.0)
- moved RIN3 0.50 mm to (71.0, 43.5)
Routing:
- net N$32: track 0.00 -> 131.7 mm, vias 0 -> 4
- net N$35: track 0.00 -> 130.5 mm, vias 0 -> 5
- net E_OVSAMP1: track 0.00 -> 125.9 mm, vias 0 -> 3
- net E_OVSAMP2: track 0.00 -> 123.8 mm, vias 0 -> 3
- net N$11: track 0.00 -> 121.3 mm, vias 0 -> 5
- net N$21: track 0.00 -> 114.1 mm, vias 0 -> 4
- net E_GSW2: track 0.00 -> 112.4 mm, vias 0 -> 5
- net E_GSW3: track 0.00 -> 110.0 mm, vias 0 -> 6
- net E_GSW4: track 0.00 -> 104.0 mm, vias 0 -> 5
- net E_SUPER1: track 0.00 -> 101.8 mm, vias 0 -> 2
- net E_GSW1: track 0.00 -> 99.4 mm, vias 0 -> 2
- net L21_SDA: track 0.00 -> 98.7 mm, vias 0 -> 5
- net E_TERM2: track 0.00 -> 93.4 mm, vias 0 -> 3
- net E_TERM4: track 0.00 -> 92.9 mm, vias 0 -> 2
- net E_SUPER4: track 0.00 -> 92.9 mm, vias 0 -> 3
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