File: eagle/max10adc dpdt.sch (EAGLE design)
At the start: 205 parts, among them IC1 MAX19506, IC2 MAX19506, J1 MOLEX_BNC_73100-0105, J2 MOLEX_BNC_73100-0105, J3 MOLEX_BNC_73100-0105, J4 MOLEX_BNC_73100-0105, K1 AQY21SOP, K2 AQY21SOP, K3 AQY21SOP, K4 AQY21SOP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

Commit message: dpdt
Changed lines of the file:
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@@
 <wire x1="-226.06" y1="-88.9" x2="-226.06" y2="-83.82" width="0.1524" layer="91"/>
 <junction x="-233.68" y="-88.9"/>
+<label x="-226.06" y="-88.9" size="1.778" layer="95" rot="R90"/>
 </segment>
 </net>
@@
 <pinref part="ST2" gate="G$1" pin="2"/>
 <wire x1="-193.04" y1="-88.9" x2="-193.04" y2="-83.82" width="0.1524" layer="91"/>
+<label x="-193.04" y="-88.9" size="1.778" layer="95" rot="R90"/>
 </segment>
 </net>
@@
 <pinref part="ST3" gate="G$1" pin="2"/>
 <wire x1="-160.02" y1="-88.9" x2="-160.02" y2="-83.82" width="0.1524" layer="91"/>
+<label x="-160.02" y="-88.9" size="1.778" layer="95" rot="R90"/>
 </segment>
 </net>
@@
 <pinref part="ST4" gate="G$1" pin="2"/>
 <wire x1="-129.54" y1="-88.9" x2="-129.54" y2="-83.82" width="0.1524" layer="91"/>
-</segment>
-</net>
+<label x="-129.54" y="-88.9" size="1.778" layer="95" rot="R90"/>
+</segment>
+</net>
