File: eagle/max10adc.sch (EAGLE design)
At the start: 205 parts, among them IC1 MAX19506, IC2 MAX19506, J1 MOLEX_BNC_73100-0105, J2 MOLEX_BNC_73100-0105, J3 MOLEX_BNC_73100-0105, J4 MOLEX_BNC_73100-0105, K1 AQY21SOP, K2 AQY21SOP, K3 AQY21SOP, K4 AQY21SOP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

Commit message: oshw logo
Parts:
- added GOLD_ORB_SM1: OSHWLOGOLOGO8MM, oshw:OSHWLOGOLOGO8MM
Changed lines of the file:
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@@
 <?xml version="1.0" encoding="utf-8"?>
 <!DOCTYPE eagle SYSTEM "eagle.dtd">
-<eagle version="8.4.3">
+<eagle version="8.6.1">
 <drawing>
 <settings>
-<setting alwaysvectorfont="yes"/>
+<setting alwaysvectorfont="no"/>
 <setting keepoldvectorfont="yes"/>
 <setting verticaltext="up"/>
@@
 <attribute name="MPN" value="06035A560FAT2A"/>
 </part>
+<part name="GOLD_ORB_SM1" library="oshw" deviceset="OSHWLOGO" device="LOGO8MM"/>
 </parts>
 <sheets>
@@
 <attribute name="MPN" x="-125.73" y="-142.24" size="1.778" layer="96" display="off"/>
 </instance>
+<instance part="GOLD_ORB_SM1" gate="G$1" x="-556.26" y="-198.12"/>
 </instances>
 <busses>
@@
 </drawing>
 <compatibility>
+<note version="6.3" minversion="6.2.2" severity="warning">
+Since Version 6.2.2 text objects can contain more than one line,
+which will not be processed correctly with this version.
+</note>
 <note version="8.2" severity="warning">
 Since Version 8.2, EAGLE supports online libraries. The ids
