File: eagle/max10adc_v9.0.brd (EAGLE design)
At the start: 98 x 79 mm, 198 parts, among them IC1 MAX19506, IC2 MAX19506, J1 MOLEX_BNC_73100-0105, J2 MOLEX_BNC_73100-0105, J3 MOLEX_BNC_73100-0105, J4 MOLEX_BNC_73100-0105, K1 AQY21SOP, K2 AQY21SOP, K3 AQY21SOP, K4 AQY21SOP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

Commit message: Cleanup schematic. Fit pages to A3. Replaces some SMD resistor so all resistor symbols are the same
Parts:
- R10M_1, R10M_2, R10M_3, R10M_4, R50-1, R50-10, R50-11, R50-12, R50-13, R50-14, R50-15, R50-16, R50-2, R50-3, R50-4, R50-5, R50-6, R50-7, R50-8, R50-9, ROFFSET1, ROFFSET2, ROFFSET3, ROFFSET4: device rcl@1:R0805 -> resistor:R0805
Changed lines of the file:
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@@
 <?xml version="1.0" encoding="utf-8"?>
 <!DOCTYPE eagle SYSTEM "eagle.dtd">
-<eagle version="9.0.1">
+<eagle version="9.1.3">
 <drawing>
 <settings>
@@
 <param name="checkStop" value="0"/>
 <param name="checkValues" value="0"/>
+<param name="checkNames" value="1"/>
+<param name="checkWireStubs" value="1"/>
+<param name="checkPolygonWidth" value="0"/>
 <param name="useDiameter" value="13"/>
 <param name="maxErrors" value="999999"/>
@@
 <attribute name="MPN" value="SN74LVC1G3157DBV" x="60" y="0.8" size="1.778" layer="27" rot="R180" display="off"/>
 </element>
-<element name="R10M_1" library="rcl@1" package="R0805" value="10M" x="83.5" y="4.8" smashed="yes" rot="R270">
+<element name="R10M_1" library="resistor" library_urn="urn:adsk.eagle:library:348" package="R0805" package3d_urn="urn:adsk.eagle:package:26059/1" value="10M" x="83.5" y="4.8" smashed="yes" rot="R270">
 <attribute name="VALUE" x="84.835" y="7.74" size="0.8128" layer="21" font="vector" rot="R180"/>
 </element>
@@
 <attribute name="VALUE" x="49.1" y="53.5" size="0.8128" layer="22" font="vector" rot="MR270"/>
 </element>
-<element name="R10M_2" library="rcl@1" package="R0805" value="10M" x="83.5" y="4.8" smashed="yes" rot="MR90">
+<element name="R10M_2" library="resistor" library_urn="urn:adsk.eagle:library:348" package="R0805" package3d_urn="urn:adsk.eagle:package:26059/1" value="10M" x="83.5" y="4.8" smashed="yes" rot="MR90">
 <attribute name="VALUE" x="84.235" y="1.56" size="0.8128" layer="22" font="vector" rot="MR0"/>
 </element>
-<element name="R10M_3" library="rcl@1" package="R0805" value="10M" x="82.4" y="46.6" smashed="yes" rot="R270">
+<element name="R10M_3" library="resistor" library_urn="urn:adsk.eagle:library:348" package="R0805" package3d_urn="urn:adsk.eagle:package:26059/1" value="10M" x="82.4" y="46.6" smashed="yes" rot="R270">
 <attribute name="VALUE" x="81.365" y="48.76" size="0.8128" layer="21" font="vector"/>
 </element>
-<element name="R10M_4" library="rcl@1" package="R0805" value="10M" x="82.4" y="46.6" smashed="yes" rot="MR270">
+<element name="R10M_4" library="resistor" library_urn="urn:adsk.eagle:library:348" package="R0805" package3d_urn="urn:adsk.eagle:package:26059/1" value="10M" x="82.4" y="46.6" smashed="yes" rot="MR270">
 <attribute name="VALUE" x="83.235" y="43.46" size="0.8128" layer="22" font="vector" rot="MR0"/>
 </element>
@@
 <attribute name="OC_NEWARK" value="unknown" x="15" y="17.7" size="0.8128" layer="27" font="vector" display="off"/>
 </element>
-<element name="R50-4" library="rcl@1" package="R0805" value="200" x="68.1" y="-8.5" smashed="yes" rot="MR0"/>
-<element name="R50-3" library="rcl@1" package="R0805" value="200" x="68.1" y="-6.4" smashed="yes" rot="MR0"/>
-<element name="R50-2" library="rcl@1" package="R0805" value="200" x="63.9" y="-6.4" smashed="yes" rot="MR0"/>
-<element name="R50-1" library="rcl@1" package="R0805" value="200" x="63.9" y="-8.5" smashed="yes" rot="MR0"/>
-<element name="R50-5" library="rcl@1" package="R0805" value="200" x="69.6" y="20.6" smashed="yes" rot="MR0"/>
-<element name="R50-6" library="rcl@1" package="R0805" value="200" x="74" y="22.8" smashed="yes" rot="MR0"/>
-<element name="R50-7" library="rcl@1" package="R0805" value="200" x="69.6" y="22.8" smashed="yes" rot="MR0"/>
-<element name="R50-8" library="rcl@1" package="R0805" value="200" x="74" y="20.6" smashed="yes" rot="MR0"/>
-<element name="R50-9" library="rcl@1" package="R0805" value="200" x="70.1" y="32.3" smashed="yes" rot="MR0"/>
-<element name="R50-10" library="rcl@1" package="R0805" value="200" x="74.3" y="32.3" smashed="yes" rot="MR0"/>
-<element name="R50-11" library="rcl@1" package="R0805" value="200" x="74.3" y="34.5" smashed="yes" rot="MR0"/>
-<element name="R50-12" library="rcl@1" package="R0805" value="200" x="70.1" y="34.5" smashed="yes" rot="MR0"/>
-<element name="R50-13" library="rcl@1" package="R0805" value="200" x="63.7" y="62.7" smashed="yes" rot="MR0"/>
-<element name="R50-14" library="rcl@1" package="R0805" value="200" x="63.7" y="60.6" smashed="yes" rot="MR0"/>
-<element name="R50-15" library="rcl@1" package="R0805" value="200" x="67.9" y="60.6" smashed="yes" rot="MR0"/>
-<element name="R50-16" library="rcl@1" package="R0805" value="200" x="67.9" y="62.7" smashed="yes" rot="MR0"/>
+<element name="R50-4" library="resistor" library_urn="urn:adsk.eagle:library:348" package="R0805" package3d_urn="urn:adsk.eagle:package:26059/1" value="200" x="68.1" y="-8.5" smashed="yes" rot="MR0"/>
+<element name="R50-3" library="resistor" library_urn="urn:adsk.eagle:library:348" package="R0805" package3d_urn="urn:adsk.eagle:package:26059/1" value="200" x="68.1" y="-6.4" smashed="yes" rot="MR0"/>
+<element name="R50-2" library="resistor" library_urn="urn:adsk.eagle:library:348" package="R0805" package3d_urn="urn:adsk.eagle:package:26059/1" value="200" x="63.9" y="-6.4" smashed="yes" rot="MR0"/>
+<element name="R50-1" library="resistor" library_urn="urn:adsk.eagle:library:348" package="R0805" package3d_urn="urn:adsk.eagle:package:26059/1" value="200" x="63.9" y="-8.5" smashed="yes" rot="MR0"/>
+<element name="R50-5" library="resistor" library_urn="urn:adsk.eagle:library:348" package="R0805" package3d_urn="urn:adsk.eagle:package:26059/1" value="200" x="69.6" y="20.6" smashed="yes" rot="MR0"/>
+<element name="R50-6" library="resistor" library_urn="urn:adsk.eagle:library:348" package="R0805" package3d_urn="urn:adsk.eagle:package:26059/1" value="200" x="74" y="22.8" smashed="yes" rot="MR0"/>
+<element name="R50-7" library="resistor" library_urn="urn:adsk.eagle:library:348" package="R0805" package3d_urn="urn:adsk.eagle:package:26059/1" value="200" x="69.6" y="22.8" smashed="yes" rot="MR0"/>
+<element name="R50-8" library="resistor" library_urn="urn:adsk.eagle:library:348" package="R0805" package3d_urn="urn:adsk.eagle:package:26059/1" value="200" x="74" y="20.6" smashed="yes" rot="MR0"/>
+<element name="R50-9" library="resistor" library_urn="urn:adsk.eagle:library:348" package="R0805" package3d_urn="urn:adsk.eagle:package:26059/1" value="200" x="70.1" y="32.3" smashed="yes" rot="MR0"/>
+<element name="R50-10" library="resistor" library_urn="urn:adsk.eagle:library:348" package="R0805" package3d_urn="urn:adsk.eagle:package:26059/1" value="200" x="74.3" y="32.3" smashed="yes" rot="MR0"/>
+<element name="R50-11" library="resistor" library_urn="urn:adsk.eagle:library:348" package="R0805" package3d_urn="urn:adsk.eagle:package:26059/1" value="200" x="74.3" y="34.5" smashed="yes" rot="MR0"/>
+<element name="R50-12" library="resistor" library_urn="urn:adsk.eagle:library:348" package="R0805" package3d_urn="urn:adsk.eagle:package:26059/1" value="200" x="70.1" y="34.5" smashed="yes" rot="MR0"/>
+<element name="R50-13" library="resistor" library_urn="urn:adsk.eagle:library:348" package="R0805" package3d_urn="urn:adsk.eagle:package:26059/1" value="200" x="63.7" y="62.7" smashed="yes" rot="MR0"/>
+<element name="R50-14" library="resistor" library_urn="urn:adsk.eagle:library:348" package="R0805" package3d_urn="urn:adsk.eagle:package:26059/1" value="200" x="63.7" y="60.6" smashed="yes" rot="MR0"/>
+<element name="R50-15" library="resistor" library_urn="urn:adsk.eagle:library:348" package="R0805" package3d_urn="urn:adsk.eagle:package:26059/1" value="200" x="67.9" y="60.6" smashed="yes" rot="MR0"/>
+<element name="R50-16" library="resistor" library_urn="urn:adsk.eagle:library:348" package="R0805" package3d_urn="urn:adsk.eagle:package:26059/1" value="200" x="67.9" y="62.7" smashed="yes" rot="MR0"/>
 <element name="U340G" library="usb-serial" package="SOIC16" value="CH340G" x="7" y="55" smashed="yes" rot="R180"/>
 <element name="Y1" library="SparkFun-FreqCtrl" package="HC49US" value="ABL-12.000MHZ-B2" x="-1.5" y="54.6" smashed="yes" rot="R90"/>
@@
 <attribute name="VALUE" x="55.8" y="0.5" size="0.8128" layer="22" font="vector" rot="MR90"/>
 </element>
-<element name="ROFFSET1" library="rcl@1" package="R0805" value="200" x="65.3" y="26.7" smashed="yes" rot="MR180">
+<element name="ROFFSET1" library="resistor" library_urn="urn:adsk.eagle:library:348" package="R0805" package3d_urn="urn:adsk.eagle:package:26059/1" value="200" x="65.3" y="26.7" smashed="yes" rot="MR180">
 <attribute name="VALUE" x="64.265" y="25.54" size="0.8128" layer="22" font="vector" rot="MR180"/>
 </element>
-<element name="ROFFSET2" library="rcl@1" package="R0805" value="200" x="65.3" y="28.9" smashed="yes" rot="MR180"/>
-<element name="ROFFSET3" library="rcl@1" package="R0805" value="200" x="65.3" y="31.1" smashed="yes" rot="MR180"/>
-<element name="ROFFSET4" library="rcl@1" package="R0805" value="200" x="65.3" y="33.3" smashed="yes" rot="MR180"/>
+<element name="ROFFSET2" library="resistor" library_urn="urn:adsk.eagle:library:348" package="R0805" package3d_urn="urn:adsk.eagle:package:26059/1" value="200" x="65.3" y="28.9" smashed="yes" rot="MR180"/>
+<element name="ROFFSET3" library="resistor" library_urn="urn:adsk.eagle:library:348" package="R0805" package3d_urn="urn:adsk.eagle:package:26059/1" value="200" x="65.3" y="31.1" smashed="yes" rot="MR180"/>
+<element name="ROFFSET4" library="resistor" library_urn="urn:adsk.eagle:library:348" package="R0805" package3d_urn="urn:adsk.eagle:package:26059/1" value="200" x="65.3" y="33.3" smashed="yes" rot="MR180"/>
 <element name="L2" library="SparkFun-Passives" package="1210" value="10uH" x="41.6" y="4" smashed="yes" rot="MR90">
 <attribute name="MPN" value="MF-IND-1210-10uH" x="41.6" y="4" size="0.8128" layer="28" font="vector" rot="MR90" display="off"/>
@@
 </signal>
 </signals>
+<mfgpreviewcolors>
+<mfgpreviewcolor name="soldermaskcolor" color="0xC8008000"/>
+<mfgpreviewcolor name="silkscreencolor" color="0xFFFEFEFE"/>
+<mfgpreviewcolor name="backgroundcolor" color="0xFF282828"/>
+<mfgpreviewcolor name="coppercolor" color="0xFFFFBF00"/>
+<mfgpreviewcolor name="substratecolor" color="0xFF786E46"/>
+</mfgpreviewcolors>
 </board>
 </drawing>

Commit message: Changed values from 200 to 200R
Parts:
- R50-1, R50-10, R50-11, R50-12, R50-13, R50-14, R50-15, R50-16, R50-2, R50-3, R50-4, R50-5, R50-6, R50-7, R50-8, R50-9, ROFFSET1, ROFFSET2, ROFFSET3, ROFFSET4: value 200 -> 200R
Changed lines of the file:
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@@
 <attribute name="OC_NEWARK" value="unknown" x="15" y="17.7" size="0.8128" layer="27" font="vector" display="off"/>
 </element>
-<element name="R50-4" library="resistor" library_urn="urn:adsk.eagle:library:348" package="R0805" package3d_urn="urn:adsk.eagle:package:26059/1" value="200" x="68.1" y="-8.5" smashed="yes" rot="MR0"/>
-<element name="R50-3" library="resistor" library_urn="urn:adsk.eagle:library:348" package="R0805" package3d_urn="urn:adsk.eagle:package:26059/1" value="200" x="68.1" y="-6.4" smashed="yes" rot="MR0"/>
-<element name="R50-2" library="resistor" library_urn="urn:adsk.eagle:library:348" package="R0805" package3d_urn="urn:adsk.eagle:package:26059/1" value="200" x="63.9" y="-6.4" smashed="yes" rot="MR0"/>
-<element name="R50-1" library="resistor" library_urn="urn:adsk.eagle:library:348" package="R0805" package3d_urn="urn:adsk.eagle:package:26059/1" value="200" x="63.9" y="-8.5" smashed="yes" rot="MR0"/>
-<element name="R50-5" library="resistor" library_urn="urn:adsk.eagle:library:348" package="R0805" package3d_urn="urn:adsk.eagle:package:26059/1" value="200" x="69.6" y="20.6" smashed="yes" rot="MR0"/>
-<element name="R50-6" library="resistor" library_urn="urn:adsk.eagle:library:348" package="R0805" package3d_urn="urn:adsk.eagle:package:26059/1" value="200" x="74" y="22.8" smashed="yes" rot="MR0"/>
-<element name="R50-7" library="resistor" library_urn="urn:adsk.eagle:library:348" package="R0805" package3d_urn="urn:adsk.eagle:package:26059/1" value="200" x="69.6" y="22.8" smashed="yes" rot="MR0"/>
-<element name="R50-8" library="resistor" library_urn="urn:adsk.eagle:library:348" package="R0805" package3d_urn="urn:adsk.eagle:package:26059/1" value="200" x="74" y="20.6" smashed="yes" rot="MR0"/>
-<element name="R50-9" library="resistor" library_urn="urn:adsk.eagle:library:348" package="R0805" package3d_urn="urn:adsk.eagle:package:26059/1" value="200" x="70.1" y="32.3" smashed="yes" rot="MR0"/>
-<element name="R50-10" library="resistor" library_urn="urn:adsk.eagle:library:348" package="R0805" package3d_urn="urn:adsk.eagle:package:26059/1" value="200" x="74.3" y="32.3" smashed="yes" rot="MR0"/>
-<element name="R50-11" library="resistor" library_urn="urn:adsk.eagle:library:348" package="R0805" package3d_urn="urn:adsk.eagle:package:26059/1" value="200" x="74.3" y="34.5" smashed="yes" rot="MR0"/>
-<element name="R50-12" library="resistor" library_urn="urn:adsk.eagle:library:348" package="R0805" package3d_urn="urn:adsk.eagle:package:26059/1" value="200" x="70.1" y="34.5" smashed="yes" rot="MR0"/>
-<element name="R50-13" library="resistor" library_urn="urn:adsk.eagle:library:348" package="R0805" package3d_urn="urn:adsk.eagle:package:26059/1" value="200" x="63.7" y="62.7" smashed="yes" rot="MR0"/>
-<element name="R50-14" library="resistor" library_urn="urn:adsk.eagle:library:348" package="R0805" package3d_urn="urn:adsk.eagle:package:26059/1" value="200" x="63.7" y="60.6" smashed="yes" rot="MR0"/>
-<element name="R50-15" library="resistor" library_urn="urn:adsk.eagle:library:348" package="R0805" package3d_urn="urn:adsk.eagle:package:26059/1" value="200" x="67.9" y="60.6" smashed="yes" rot="MR0"/>
-<element name="R50-16" library="resistor" library_urn="urn:adsk.eagle:library:348" package="R0805" package3d_urn="urn:adsk.eagle:package:26059/1" value="200" x="67.9" y="62.7" smashed="yes" rot="MR0"/>
+<element name="R50-4" library="resistor" library_urn="urn:adsk.eagle:library:348" package="R0805" package3d_urn="urn:adsk.eagle:package:26059/1" value="200R" x="68.1" y="-8.5" smashed="yes" rot="MR0"/>
+<element name="R50-3" library="resistor" library_urn="urn:adsk.eagle:library:348" package="R0805" package3d_urn="urn:adsk.eagle:package:26059/1" value="200R" x="68.1" y="-6.4" smashed="yes" rot="MR0"/>
+<element name="R50-2" library="resistor" library_urn="urn:adsk.eagle:library:348" package="R0805" package3d_urn="urn:adsk.eagle:package:26059/1" value="200R" x="63.9" y="-6.4" smashed="yes" rot="MR0"/>
+<element name="R50-1" library="resistor" library_urn="urn:adsk.eagle:library:348" package="R0805" package3d_urn="urn:adsk.eagle:package:26059/1" value="200R" x="63.9" y="-8.5" smashed="yes" rot="MR0"/>
+<element name="R50-5" library="resistor" library_urn="urn:adsk.eagle:library:348" package="R0805" package3d_urn="urn:adsk.eagle:package:26059/1" value="200R" x="69.6" y="20.6" smashed="yes" rot="MR0"/>
+<element name="R50-6" library="resistor" library_urn="urn:adsk.eagle:library:348" package="R0805" package3d_urn="urn:adsk.eagle:package:26059/1" value="200R" x="74" y="22.8" smashed="yes" rot="MR0"/>
+<element name="R50-7" library="resistor" library_urn="urn:adsk.eagle:library:348" package="R0805" package3d_urn="urn:adsk.eagle:package:26059/1" value="200R" x="69.6" y="22.8" smashed="yes" rot="MR0"/>
+<element name="R50-8" library="resistor" library_urn="urn:adsk.eagle:library:348" package="R0805" package3d_urn="urn:adsk.eagle:package:26059/1" value="200R" x="74" y="20.6" smashed="yes" rot="MR0"/>
+<element name="R50-9" library="resistor" library_urn="urn:adsk.eagle:library:348" package="R0805" package3d_urn="urn:adsk.eagle:package:26059/1" value="200R" x="70.1" y="32.3" smashed="yes" rot="MR0"/>
+<element name="R50-10" library="resistor" library_urn="urn:adsk.eagle:library:348" package="R0805" package3d_urn="urn:adsk.eagle:package:26059/1" value="200R" x="74.3" y="32.3" smashed="yes" rot="MR0"/>
+<element name="R50-11" library="resistor" library_urn="urn:adsk.eagle:library:348" package="R0805" package3d_urn="urn:adsk.eagle:package:26059/1" value="200R" x="74.3" y="34.5" smashed="yes" rot="MR0"/>
+<element name="R50-12" library="resistor" library_urn="urn:adsk.eagle:library:348" package="R0805" package3d_urn="urn:adsk.eagle:package:26059/1" value="200R" x="70.1" y="34.5" smashed="yes" rot="MR0"/>
+<element name="R50-13" library="resistor" library_urn="urn:adsk.eagle:library:348" package="R0805" package3d_urn="urn:adsk.eagle:package:26059/1" value="200R" x="63.7" y="62.7" smashed="yes" rot="MR0"/>
+<element name="R50-14" library="resistor" library_urn="urn:adsk.eagle:library:348" package="R0805" package3d_urn="urn:adsk.eagle:package:26059/1" value="200R" x="63.7" y="60.6" smashed="yes" rot="MR0"/>
+<element name="R50-15" library="resistor" library_urn="urn:adsk.eagle:library:348" package="R0805" package3d_urn="urn:adsk.eagle:package:26059/1" value="200R" x="67.9" y="60.6" smashed="yes" rot="MR0"/>
+<element name="R50-16" library="resistor" library_urn="urn:adsk.eagle:library:348" package="R0805" package3d_urn="urn:adsk.eagle:package:26059/1" value="200R" x="67.9" y="62.7" smashed="yes" rot="MR0"/>
 <element name="U340G" library="usb-serial" package="SOIC16" value="CH340G" x="7" y="55" smashed="yes" rot="R180"/>
 <element name="Y1" library="SparkFun-FreqCtrl" package="HC49US" value="ABL-12.000MHZ-B2" x="-1.5" y="54.6" smashed="yes" rot="R90"/>
@@
 <attribute name="VALUE" x="55.8" y="0.5" size="0.8128" layer="22" font="vector" rot="MR90"/>
 </element>
-<element name="ROFFSET1" library="resistor" library_urn="urn:adsk.eagle:library:348" package="R0805" package3d_urn="urn:adsk.eagle:package:26059/1" value="200" x="65.3" y="26.7" smashed="yes" rot="MR180">
+<element name="ROFFSET1" library="resistor" library_urn="urn:adsk.eagle:library:348" package="R0805" package3d_urn="urn:adsk.eagle:package:26059/1" value="200R" x="65.3" y="26.7" smashed="yes" rot="MR180">
 <attribute name="VALUE" x="64.265" y="25.54" size="0.8128" layer="22" font="vector" rot="MR180"/>
 </element>
-<element name="ROFFSET2" library="resistor" library_urn="urn:adsk.eagle:library:348" package="R0805" package3d_urn="urn:adsk.eagle:package:26059/1" value="200" x="65.3" y="28.9" smashed="yes" rot="MR180"/>
-<element name="ROFFSET3" library="resistor" library_urn="urn:adsk.eagle:library:348" package="R0805" package3d_urn="urn:adsk.eagle:package:26059/1" value="200" x="65.3" y="31.1" smashed="yes" rot="MR180"/>
-<element name="ROFFSET4" library="resistor" library_urn="urn:adsk.eagle:library:348" package="R0805" package3d_urn="urn:adsk.eagle:package:26059/1" value="200" x="65.3" y="33.3" smashed="yes" rot="MR180"/>
+<element name="ROFFSET2" library="resistor" library_urn="urn:adsk.eagle:library:348" package="R0805" package3d_urn="urn:adsk.eagle:package:26059/1" value="200R" x="65.3" y="28.9" smashed="yes" rot="MR180"/>
+<element name="ROFFSET3" library="resistor" library_urn="urn:adsk.eagle:library:348" package="R0805" package3d_urn="urn:adsk.eagle:package:26059/1" value="200R" x="65.3" y="31.1" smashed="yes" rot="MR180"/>
+<element name="ROFFSET4" library="resistor" library_urn="urn:adsk.eagle:library:348" package="R0805" package3d_urn="urn:adsk.eagle:package:26059/1" value="200R" x="65.3" y="33.3" smashed="yes" rot="MR180"/>
 <element name="L2" library="SparkFun-Passives" package="1210" value="10uH" x="41.6" y="4" smashed="yes" rot="MR90">
 <attribute name="MPN" value="MF-IND-1210-10uH" x="41.6" y="4" size="0.8128" layer="28" font="vector" rot="MR90" display="off"/>

Commit message: clean up a few things
Parts:
- turned S1 to 0 degrees
- turned S5 to 0 degrees
Connections:
- net N$20 renamed NSG_1
- net N$24 renamed N10M_1
- net N$29 renamed N50_1
- net N$37 renamed NNG_1
Routing:
- net GND: track 273.7 -> 234.7 mm
- net N$11: track 98.7 -> 111.2 mm, vias 4 -> 6
- net N$10: track 42.6 -> 31.1 mm, vias 2 -> 1
- net NSG_1: track 12.6 -> 20.1 mm
- net N10M_1: track 19.3 -> 25.7 mm
- net NNG_1: track 42.3 -> 37.9 mm, vias 1 -> 2
- net +3V3: track 382.3 -> 378.0 mm
- net N50_1: track 14.5 -> 10.9 mm
- net D5B: track 19.5 -> 16.1 mm
- net INJ1: track 22.1 -> 24.6 mm, vias 3 -> 2
- net E_21_B4: track 103.6 -> 105.8 mm
- net N$35: track 163.5 -> 161.7 mm
- net D1A: track 16.5 -> 15.0 mm
- net E_GSW1: track 116.9 -> 115.4 mm
- net E_21_B0: track 93.8 -> 94.8 mm
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Other:
- board text added: "Super gain"
- board text removed: "Normal gain"
