File: eagle/max10adc_v9.0_16chan_frontendtest2.brd (EAGLE design)
At the start: 170 x 79 mm, 182 parts, among them IC1 MAX11115AUT+T, IC2 MAX11115AUT+T, IC3 MAX11115AUT+T, IC4 MAX11115AUT+T, K1 AQY21SOP, K3 AQY21SOP, K5 AQY21SOP, K6 AQY21SOP, U340G CH340G, X1 LTI-SASF54GT, X4 LTI-SASF54GT, X5 LTI-SASF54GT, X6 LTI-SASF54GT, Y1 ABL-12.000MHZ-B2

Commit message: routed for MF
Parts:
- added ACR10, ACR11, ACR12, ACR13, ACR14, ACR15, ACR16, ACR21, ACR22, ACR23, ACR24, ACR9: 560, resistor:R0805
- added BJ2, BJ3, BJ4: 6p-2.54, Seeed-Connector:H6-2.54
- added C5VOPAMP3, C5VOPAMP4, C5VOPAMP6, CADD10, CADD11, CADD12, CADD13, CADD14, CADD15, CADD16, CADD21, CADD22, CADD23, CADD24, CADD9, COB10, COB11, COB12, COB13, COB14, COB15, COB16, COB21, COB22, COB23, COB24, COB9, COFFSET2, COFFSET3, COFFSET5: 0.1uF, rcl:C0805K
- added CAC10, CAC11, CAC12, CAC13, CAC14, CAC15, CAC16, CAC21, CAC22, CAC23, CAC24, CAC9: 0.01uF, rcl@1:C0603
- added CGAIN1_10, CGAIN1_11, CGAIN1_12, CGAIN1_13, CGAIN1_14, CGAIN1_15, CGAIN1_16, CGAIN1_21, CGAIN1_22, CGAIN1_23, CGAIN1_24, CGAIN1_9: 220pF, rcl@1:C0603
- added CH10, CH11, CH12, CH13, CH14, CH15, CH16, CH2, CH4, CH7, CH8, CH9, CL10, CL11, CL12, CL13, CL14, CL15, CL16, CL2, CL4, CL7, CL8, CL9: 8-45pF, SparkFun-Passives:CTZ3
- added CIN10, CIN11, CIN12, CIN13, CIN14, CIN15, CIN16, CIN21, CIN22, CIN23, CIN24, CIN9: 10pF, rcl@1:C0603
- added CIN56S10, CIN56S11, CIN56S12, CIN56S13, CIN56S14, CIN56S15, CIN56S16, CIN56S21, CIN56S22, CIN56S23, CIN56S24, CIN56S9: 56pF, rcl@1:C0603
- added CINS10, CINS11, CINS12, CINS13, CINS14, CINS15, CINS16, CINS21, CINS22, CINS23, CINS24, CINS9: 1nF, rcl@1:C0603
- added COA10, COA11, COA12, COA13, COA14, COA15, COA16, COA21, COA22, COA23, COA24, COA9: 10uF, rcl@1:C1206
- added DAC2, DAC3, DAC4: MCP4728, Luca Eagle-Library:MSOP10
- added GSW10, GSW11, GSW12, GSW13, GSW14, GSW15, GSW16, GSW21, GSW22, GSW23, GSW24, GSW9: 741G3157DBVR, 74xx-little-us:DBV_R-PDSO-G6
- added IC10, IC11, IC12, IC13, IC14, IC15, IC16, IC21, IC22, IC23, IC24, IC9: MAX11115AUT+T, SamacSys_Parts:SOT95P280X145-6N
- added ICAMP3, ICAMP4, ICAMP6: OPA4322AIPWR, SamacSys_Parts:SOP65P640X120-16N
- added IN10, IN11, IN12, IN13, IN14, IN15, IN16, IN5, IN6, IN7, IN8, IN9: 2p-2.54, Seeed-Connector:H2-2.54
- added K10, K11, K12, K13, K14, K15, K16, K21, K22, K23, K24, K9: AQY21SOP, relay:SOP04
- added R50-33, R50-34, R50-35, R50-36, R50-37, R50-38, R50-39, R50-40, R50-41, R50-42, R50-43, R50-44, R50-45, R50-46, R50-47, R50-48, R50-49, R50-50, R50-51, R50-52, R50-53, R50-54, R50-55, R50-56, R50-57, R50-58, R50-59, R50-60, R50-61, R50-62, R50-63, R50-64, R50-81, R50-82, R50-83, R50-84, R50-85, R50-86, R50-87, R50-88, R50-89, R50-90, R50-91, R50-92, R50-93, R50-94, R50-95, R50-96: 200R, resistor:R0805
- added RG1_11, RG1_12, RG1_5, RG1_6, RG1_7, RG1_8, RG3_11, RG3_12, RG3_3, RG3_4, RG3_7, RG3_8: 47k, resistor:R0805
- added RG2_11, RG2_12, RG2_5, RG2_6, RG2_7, RG2_8, RG4_11, RG4_12, RG4_3, RG4_4, RG4_7, RG4_8: 470k, resistor:R0805
- added RIN10, RIN11, RIN12, RIN13, RIN14, RIN15, RIN16, RIN21, RIN22, RIN23, RIN24, RIN9: 1.1M, resistor:R0805
- added RIN10M10, RIN10M11, RIN10M12, RIN10M13, RIN10M14, RIN10M15, RIN10M16, RIN10M21, RIN10M22, RIN10M23, RIN10M24, RIN10M9: 10M, resistor:R0805
- added RINS10, RINS11, RINS12, RINS13, RINS14, RINS15, RINS16, RINS21, RINS22, RINS23, RINS24, RINS9: 11K, resistor:R0805
- added ROFFSET10, ROFFSET11, ROFFSET12, ROFFSET13, ROFFSET14, ROFFSET15, ROFFSET16, ROFFSET21, ROFFSET22, ROFFSET23, ROFFSET24, ROFFSET9: 200, resistor:R0805
- added S18, S19, S20, S21, S22, S23, S24, S25, S26, S27, S28, S29, S30, S31, S32, S33, S42, S43, S44, S45, S46, S47, S48, S49: JS202011SCQN, switch-ck:JS202011SCQN
- added X10, X11, X12, X13, X14, X15, X16, X21, X22, X23, X24, X9: LTI-SASF54GT, con-coax:LTI-SASF54GT
- moved CH5 10.0 mm to (83.3, 10.0)
- moved CH6 10.0 mm to (83.3, 15.0)
- moved CL5 10.0 mm to (77.0, 10.0)
- moved CL6 10.0 mm to (77.0, 15.0)
- moved R_SCL 9.22 mm to (8.00, 15.2)
- moved R_SDA 9.22 mm to (8.00, 13.0)
- moved CH3 5.00 mm to (83.3, 0.00), flipped to the top, turned to 270 degrees
- moved CL3 5.00 mm to (77.0, 0.00), flipped to the top, turned to 270 degrees
- moved ROFFSET1 3.00 mm to (59.3, -8.90), flipped to the bottom
- moved ROFFSET2 3.00 mm to (63.7, -8.90), flipped to the bottom
- moved ROFFSET4 3.00 mm to (59.2, 3.90), flipped to the bottom
- moved ROFFSET3 3.00 mm to (63.6, 3.80), flipped to the bottom
- moved COA1 2.00 mm to (66.6, -9.40)
- moved COA2 2.00 mm to (66.5, 4.30)
- moved COB2 2.00 mm to (64.5, 3.80)
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- renumbered RLEDPOW to RPOW
Connections:
- new net CGAIN17: CGAIN1_9.2, CL5.-, GSW9.3, RG1_5.1
- new net CGAIN18: CH5.-, GSW9.1, RG2_5.1
- new net CGAIN19: CGAIN1_10.2, CL6.-, GSW10.3, RG1_6.1
- new net CGAIN20: CH6.-, GSW10.1, RG2_6.1
- new net CGAIN21: CGAIN1_11.2, CL7.-, GSW11.3, RG3_3.1
- new net CGAIN22: CH7.-, GSW11.1, RG4_3.1
- new net CGAIN23: CGAIN1_12.2, CL8.-, GSW12.3, RG3_4.1
- new net CGAIN24: CH8.-, GSW12.1, RG4_4.1
- new net CGAIN25: CGAIN1_13.2, CL9.-, GSW13.3, RG1_7.1
- new net CGAIN26: CH9.-, GSW13.1, RG2_7.1
- new net CGAIN27: CGAIN1_14.2, CL10.-, GSW14.3, RG1_8.1
- new net CGAIN28: CH10.-, GSW14.1, RG2_8.1
- new net CGAIN29: CGAIN1_15.2, CL11.-, GSW15.3, RG3_7.1
- new net CGAIN30: CH11.-, GSW15.1, RG4_7.1
- new net CGAIN31: CGAIN1_16.2, CL12.-, GSW16.3, RG3_8.1
- new net CGAIN32: CH12.-, GSW16.1, RG4_8.1
- new net CGAIN41: CGAIN1_21.2, CL13.-, GSW21.3, RG1_11.1
- new net CGAIN42: CH13.-, GSW21.1, RG2_11.1
- new net CGAIN43: CGAIN1_22.2, CL14.-, GSW22.3, RG1_12.1
- new net CGAIN44: CH14.-, GSW22.1, RG2_12.1
- new net CGAIN45: CGAIN1_23.2, CL15.-, GSW23.3, RG3_11.1
- new net CGAIN46: CH15.-, GSW23.1, RG4_11.1
- new net CGAIN47: CGAIN1_24.2, CL16.-, GSW24.3, RG3_12.1
- new net CGAIN48: CH16.-, GSW24.1, RG4_12.1
- new net INA10: GSW14.4, IC15.3, ICAMP4.7
- new net INA11: GSW15.4, IC16.3, ICAMP4.10
- new net INA12: GSW16.4, IC13.3, ICAMP4.16
- new net INA13: GSW21.4, IC22.3, ICAMP6.1
- new net INA14: GSW22.4, IC23.3, ICAMP6.7
- new net INA15: GSW23.4, IC24.3, ICAMP6.10
- new net INA16: GSW24.4, IC21.3, ICAMP6.16
- new net INA5: GSW9.4, IC10.3, ICAMP3.1
- new net INA6: GSW10.4, IC11.3, ICAMP3.7
- new net INA7: GSW11.4, IC12.3, ICAMP3.10
- new net INA8: GSW12.4, IC9.3, ICAMP3.16
- new net INA9: GSW13.4, IC14.3, ICAMP4.1
- new net INAMINUS10: CGAIN1_14.1, CH10.+, CIN14.2, CIN56S14.2, CINS14.2, CL10.+, ICAMP4.6, RG1_8.2, RG2_8.2, RIN14.2, RINS14.2
- new net INAMINUS11: CGAIN1_15.1, CH11.+, CIN15.2, CIN56S15.2, CINS15.2, CL11.+, ICAMP4.11, RG3_7.2, RG4_7.2, RIN15.2, RINS15.2
- new net INAMINUS12: CGAIN1_16.1, CH12.+, CIN16.2, CIN56S16.2, CINS16.2, CL12.+, ICAMP4.15, RG3_8.2, RG4_8.2, RIN16.2, RINS16.2
- new net INAMINUS13: CGAIN1_21.1, CH13.+, CIN21.2, CIN56S21.2, CINS21.2, CL13.+, ICAMP6.2, RG1_11.2, RG2_11.2, RIN21.2, RINS21.2
- new net INAMINUS14: CGAIN1_22.1, CH14.+, CIN22.2, CIN56S22.2, CINS22.2, CL14.+, ICAMP6.6, RG1_12.2, RG2_12.2, RIN22.2, RINS22.2
- new net INAMINUS15: CGAIN1_23.1, CH15.+, CIN23.2, CIN56S23.2, CINS23.2, CL15.+, ICAMP6.11, RG3_11.2, RG4_11.2, RIN23.2, RINS23.2
- new net INAMINUS16: CGAIN1_24.1, CH16.+, CIN24.2, CIN56S24.2, CINS24.2, CL16.+, ICAMP6.15, RG3_12.2, RG4_12.2, RIN24.2, RINS24.2
- new net INAMINUS5: CGAIN1_9.1, CH5.+, CIN56S9.2, CIN9.2, CINS9.2, CL5.+, ICAMP3.2, RG1_5.2, RG2_5.2, RIN9.2, RINS9.2
- new net INAMINUS6: CGAIN1_10.1, CH6.+, CIN10.2, CIN56S10.2, CINS10.2, CL6.+, ICAMP3.6, RG1_6.2, RG2_6.2, RIN10.2, RINS10.2
- new net INAMINUS7: CGAIN1_11.1, CH7.+, CIN11.2, CIN56S11.2, CINS11.2, CL7.+, ICAMP3.11, RG3_3.2, RG4_3.2, RIN11.2, RINS11.2
- new net INAMINUS8: CGAIN1_12.1, CH8.+, CIN12.2, CIN56S12.2, CINS12.2, CL8.+, ICAMP3.15, RG3_4.2, RG4_4.2, RIN12.2, RINS12.2
- new net INAMINUS9: CGAIN1_13.1, CH9.+, CIN13.2, CIN56S13.2, CINS13.2, CL9.+, ICAMP4.2, RG1_7.2, RG2_7.2, RIN13.2, RINS13.2
- new net INJ10: BJ3.4, CAC14.2, IN10.2, K14.3, S28.2, X14.1
- new net INJ11: BJ3.3, CAC15.2, IN11.2, K15.3, S30.2, X15.1
- new net INJ12: BJ3.2, CAC16.2, IN12.2, K16.3, S32.2, X16.1
- new net INJ13: BJ4.5, CAC21.2, IN13.2, K21.3, S42.2, X21.1
- new net INJ14: BJ4.4, CAC22.2, IN14.2, K22.3, S44.2, X22.1
- new net INJ15: BJ4.3, CAC23.2, IN15.2, K23.3, S46.2, X23.1
- new net INJ16: BJ4.2, CAC24.2, IN16.2, K24.3, S48.2, X24.1
- new net INJ5: BJ2.5, CAC9.2, IN5.2, K9.3, S18.2, X9.1
- new net INJ6: BJ2.4, CAC10.2, IN6.2, K10.3, S20.2, X10.1
- new net INJ7: BJ2.3, CAC11.2, IN7.2, K11.3, S22.2, X11.1
- new net INJ8: BJ2.2, CAC12.2, IN8.2, K12.3, S24.2, X12.1
- new net INJ9: BJ3.5, CAC13.2, IN9.2, K13.3, S26.2, X13.1
- new net N$15: DAC2.6, ROFFSET9.2
- new net N$16: DAC2.7, ROFFSET10.2
- new net N$17: DAC2.8, ROFFSET11.2
- new net N$19: DAC2.9, ROFFSET12.2
- new net N$2: ACR11.2, K10.1
- new net N$20: DAC3.6, ROFFSET13.2
- new net N$21: DAC3.7, ROFFSET14.2
- new net N$22: DAC3.8, ROFFSET15.2
- new net N$25: DAC3.9, ROFFSET16.2
- new net N$28: CAC9.1, K9.4, RIN10M9.1, S19.2
- new net N$29: CAC10.1, K10.4, RIN10M10.1, S21.2
- new net N$3: ACR10.2, K11.1
- new net N$30: CAC11.1, K11.4, RIN10M11.1, S23.2
- new net N$32: CAC12.1, K12.4, RIN10M12.1, S25.2
- new net N$37: ACR15.2, K14.1
- new net N$38: ACR14.2, K15.1
- new net N$39: ACR16.2, K16.1
- new net N$40: ACR21.2, K21.1
- new net N$41: DAC4.6, ROFFSET21.2
- new net N$42: DAC4.7, ROFFSET22.2
- new net N$43: DAC4.8, ROFFSET23.2
- new net N$50: DAC4.9, ROFFSET24.2
- new net N$52: CAC13.1, K13.4, RIN10M13.1, S27.2
- new net N$53: CAC14.1, K14.4, RIN10M14.1, S29.2
- new net N$54: CAC15.1, K15.4, RIN10M15.1, S31.2
- new net N$55: CAC16.1, K16.4, RIN10M16.1, S33.2
- new net N$59: ACR23.2, K22.1
- new net N$60: ACR22.2, K23.1
- new net N$61: ACR24.2, K24.1
- new net N$62: ACR9.2, K9.1
- new net N$68: CAC21.1, K21.4, RIN10M21.1, S43.2
- new net N$69: CAC22.1, K22.4, RIN10M22.1, S45.2
- new net N$7: ACR12.2, K12.1
- new net N$70: CAC23.1, K23.4, RIN10M23.1, S47.2
- new net N$71: CAC24.1, K24.4, RIN10M24.1, S49.2
- new net N$8: ACR13.2, K13.1
- new net N50_10: R50-53.1, R50-54.1, R50-55.1, R50-56.1, S28.3
- new net N50_11: R50-57.1, R50-58.1, R50-59.1, R50-60.1, S30.3
- new net N50_12: R50-61.1, R50-62.1, R50-63.1, R50-64.1, S32.3
- new net N50_13: R50-81.1, R50-82.1, R50-83.1, R50-84.1, S42.3
- new net N50_14: R50-85.1, R50-86.1, R50-87.1, R50-88.1, S44.3
- new net N50_15: R50-89.1, R50-90.1, R50-91.1, R50-92.1, S46.3
- new net N50_16: R50-93.1, R50-94.1, R50-95.1, R50-96.1, S48.3
- new net N50_5: R50-33.1, R50-34.1, R50-35.1, R50-36.1, S18.3
- new net N50_6: R50-37.1, R50-38.1, R50-39.1, R50-40.1, S20.3
- new net N50_7: R50-41.1, R50-42.1, R50-43.1, R50-44.1, S22.3
- new net N50_8: R50-45.1, R50-46.1, R50-47.1, R50-48.1, S24.3
- new net N50_9: R50-49.1, R50-50.1, R50-51.1, R50-52.1, S26.3
- new net NNG_10: CIN14.1, RIN14.1, S29.3
- new net NNG_11: CIN15.1, RIN15.1, S31.3
- new net NNG_12: CIN16.1, RIN16.1, S33.3
- new net NNG_13: CIN21.1, RIN21.1, S43.3
- new net NNG_14: CIN22.1, RIN22.1, S45.3
- new net NNG_15: CIN23.1, RIN23.1, S47.3
- new net NNG_16: CIN24.1, RIN24.1, S49.3
- new net NNG_5: CIN9.1, RIN9.1, S19.3
- new net NNG_6: CIN10.1, RIN10.1, S21.3
- new net NNG_7: CIN11.1, RIN11.1, S23.3
- new net NNG_8: CIN12.1, RIN12.1, S25.3
- new net NNG_9: CIN13.1, RIN13.1, S27.3
- new net NSG_10: CIN56S14.1, CINS14.1, RINS14.1, S29.1
- new net NSG_11: CIN56S15.1, CINS15.1, RINS15.1, S31.1
- new net NSG_12: CIN56S16.1, CINS16.1, RINS16.1, S33.1
- new net NSG_13: CIN56S21.1, CINS21.1, RINS21.1, S43.1
- new net NSG_14: CIN56S22.1, CINS22.1, RINS22.1, S45.1
- new net NSG_15: CIN56S23.1, CINS23.1, RINS23.1, S47.1
- new net NSG_16: CIN56S24.1, CINS24.1, RINS24.1, S49.1
- new net NSG_5: CIN56S9.1, CINS9.1, RINS9.1, S19.1
- new net NSG_6: CIN56S10.1, CINS10.1, RINS10.1, S21.1
- new net NSG_7: CIN56S11.1, CINS11.1, RINS11.1, S23.1
- new net NSG_8: CIN56S12.1, CINS12.1, RINS12.1, S25.1
- new net NSG_9: CIN56S13.1, CINS13.1, RINS13.1, S27.1
- new net OFFSET10: COA14.2, COB14.2, ICAMP4.5, ROFFSET14.1
- new net OFFSET11: COA15.2, COB15.2, ICAMP4.12, ROFFSET15.1
- new net OFFSET12: COA16.2, COB16.2, ICAMP4.14, ROFFSET16.1
- new net OFFSET13: COA21.2, COB21.2, ICAMP6.3, ROFFSET21.1
- new net OFFSET14: COA22.2, COB22.2, ICAMP6.5, ROFFSET22.1
- new net OFFSET15: COA23.2, COB23.2, ICAMP6.12, ROFFSET23.1
- new net OFFSET16: COA24.2, COB24.2, ICAMP6.14, ROFFSET24.1
- new net OFFSET5: COA9.2, COB9.2, ICAMP3.3, ROFFSET9.1
- new net OFFSET6: COA10.2, COB10.2, ICAMP3.5, ROFFSET10.1
- new net OFFSET7: COA11.2, COB11.2, ICAMP3.12, ROFFSET11.1
- new net OFFSET8: COA12.2, COB12.2, ICAMP3.14, ROFFSET12.1
- new net OFFSET9: COA13.2, COB13.2, ICAMP4.3, ROFFSET13.1
- net CGAIN10: now also CH3.-; no longer CH5.-
- net CGAIN11: now also CL4.-; no longer CL6.-
- net CGAIN12: now also CH4.-; no longer CH6.-
- net CGAIN5: now also CL2.-; no longer CL3.-
- net CGAIN6: now also CH2.-; no longer CH3.-
- net CGAIN9: now also CL3.-; no longer CL5.-
- net CLKOUT_32: now also IC10.4, IC11.4, IC12.4, IC13.4, IC14.4, IC15.4, IC16.4, IC21.4, IC22.4, IC23.4, IC24.4, IC9.4
- net CLKOUT_33: now also IC10.6, IC11.6, IC12.6, IC13.6, IC14.6, IC15.6, IC16.6, IC21.6, IC22.6, IC23.6, IC24.6, IC9.6
- net D0B: now also IC14.5
- net D1B: now also IC15.5
- net D2B: now also IC16.5
- net D3B: now also IC13.5
- net D4A: now also IC10.5
- net D4B: now also IC22.5
- net D5A: now also IC11.5
- net D5B: now also IC23.5
- net D6A: now also IC12.5
- net D6B: now also IC24.5
- net D7A: now also IC9.5
- net D7B: now also IC21.5
- net E_50SW10: now also S28.5
- net E_50SW11: now also S30.5
- net E_50SW12: now also S32.5
- net E_50SW13: now also S42.5
- net E_50SW14: now also S44.5
- net E_50SW15: now also S46.5
- net E_50SW16: now also S48.5
- net E_50SW5: now also S18.5
- net E_50SW6: now also S20.5
- net E_50SW7: now also S22.5
- net E_50SW8: now also S24.5
- net E_50SW9: now also S26.5
- net E_ACSW10: now also ACR15.1
- net E_ACSW11: now also ACR14.1
- net E_ACSW12: now also ACR16.1
- net E_ACSW13: now also ACR21.1
- net E_ACSW14: now also ACR23.1
- net E_ACSW15: now also ACR22.1
- net E_ACSW16: now also ACR24.1
- net E_ACSW5: now also ACR9.1
- net E_ACSW6: now also ACR11.1
- net E_ACSW7: now also ACR10.1
- net E_ACSW8: now also ACR12.1
- net E_ACSW9: now also ACR13.1
- net E_GSW10: now also GSW14.6
- net E_GSW11: now also GSW15.6
- net E_GSW12: now also GSW16.6
- net E_GSW13: now also GSW21.6
- net E_GSW14: now also GSW22.6
- net E_GSW15: now also GSW23.6
- net E_GSW16: now also GSW24.6
- net E_GSW5: now also GSW9.6
- net E_GSW6: now also GSW10.6
- net E_GSW7: now also GSW11.6
- net E_GSW8: now also GSW12.6
- net E_GSW9: now also GSW13.6
- net E_SS10: now also S29.5
- net E_SS11: now also S31.5
- net E_SS12: now also S33.5
- net E_SS13: now also S43.5
- net E_SS14: now also S45.5
- net E_SS15: now also S47.5
- net E_SS16: now also S49.5
- net E_SS5: now also S19.5
- net E_SS6: now also S21.5
- net E_SS7: now also S23.5
- net E_SS8: now also S25.5
- net E_SS9: now also S27.5
- net GND: now also BJ2.1, BJ3.1, BJ4.1, C5VOPAMP3.2, C5VOPAMP4.2, C5VOPAMP6.2, CADD10.2, CADD11.2, CADD12.2, CADD13.2, CADD14.2, CADD15.2, CADD16.2, CADD21.2, CADD22.2, CADD23.2, CADD24.2, CADD9.2, COA10.1, COA11.1, COA12.1, COA13.1, COA14.1, COA15.1, COA16.1, COA21.1, COA22.1, COA23.1, COA24.1, COA9.1, COB10.1, COB11.1, COB12.1, COB13.1, COB14.1, COB15.1, COB16.1, COB21.1, COB22.1, COB23.1, COB24.1, COB9.1, COFFSET2.1, COFFSET3.1, COFFSET5.1, DAC2.10, DAC2.4, DAC3.10, DAC3.4, DAC4.10, DAC4.4, GSW10.2, GSW11.2, GSW12.2, GSW13.2, GSW14.2, GSW15.2, GSW16.2, GSW21.2, GSW22.2, GSW23.2, GSW24.2, GSW9.2, IC10.2, IC11.2, IC12.2, IC13.2, IC14.2, IC15.2, IC16.2, IC21.2, IC22.2, IC23.2, IC24.2, IC9.2, ICAMP3.13, ICAMP4.13, ICAMP6.13, IN10.1, IN11.1, IN12.1, IN13.1, IN14.1, IN15.1, IN16.1, IN5.1, IN6.1, IN7.1, IN8.1, IN9.1, K10.2, K11.2, K12.2, K13.2, K14.2, K15.2, K16.2, K21.2, K22.2, K23.2, K24.2, K9.2, R50-33.2, R50-34.2, R50-35.2, R50-36.2, R50-37.2, R50-38.2, R50-39.2, R50-40.2, R50-41.2, R50-42.2, R50-43.2, R50-44.2, R50-45.2, R50-46.2, R50-47.2, R50-48.2, R50-49.2, R50-50.2, R50-51.2, R50-52.2, R50-53.2, R50-54.2, R50-55.2, R50-56.2, R50-57.2, R50-58.2, R50-59.2, R50-60.2, R50-61.2, R50-62.2, R50-63.2, R50-64.2, R50-81.2, R50-82.2, R50-83.2, R50-84.2, R50-85.2, R50-86.2, R50-87.2, R50-88.2, R50-89.2, R50-90.2, R50-91.2, R50-92.2, R50-93.2, R50-94.2, R50-95.2, R50-96.2, RIN10M10.2, RIN10M11.2, RIN10M12.2, RIN10M13.2, RIN10M14.2, RIN10M15.2, RIN10M16.2, RIN10M21.2, RIN10M22.2, RIN10M23.2, RIN10M24.2, RIN10M9.2, S18.6, S19.6, S20.6, S21.6, S22.6, S23.6, S24.6, S25.6, S26.6, S27.6, S28.6, S29.6, S30.6, S31.6, S32.6, S33.6, S42.6, S43.6, S44.6, S45.6, S46.6, S47.6, S48.6, S49.6, X10.2, X10.3, X10.4, X10.5, X11.2, X11.3, X11.4, X11.5, X12.2, X12.3, X12.4, X12.5, X13.2, X13.3, X13.4, X13.5, X14.2, X14.3, X14.4, X14.5, X15.2, X15.3, X15.4, X15.5, X16.2, X16.3, X16.4, X16.5, X21.2, X21.3, X21.4, X21.5, X22.2, X22.3, X22.4, X22.5, X23.2, X23.3, X23.4, X23.5, X24.2, X24.3, X24.4, X24.5, X9.2, X9.3, X9.4, X9.5
- net INAMINUS2: now also CH2.+, CL2.+; no longer CH3.+, CL3.+
- net INAMINUS3: now also CH3.+, CL3.+; no longer CH5.+, CL5.+
- net INAMINUS4: now also CH4.+, CL4.+; no longer CH6.+, CL6.+
- net L141_SCL: now also DAC2.2, DAC3.2, DAC4.2
- net L21_SDA: now also DAC2.3, DAC3.3, DAC4.3
- net VCCA: now also BJ2.6, BJ3.6, BJ4.6, C5VOPAMP3.1, C5VOPAMP4.1, C5VOPAMP6.1, CADD10.1, CADD11.1, CADD12.1, CADD13.1, CADD14.1, CADD15.1, CADD16.1, CADD21.1, CADD22.1, CADD23.1, CADD24.1, CADD9.1, COFFSET2.2, COFFSET3.2, COFFSET5.2, DAC2.1, DAC3.1, DAC4.1, GSW10.5, GSW11.5, GSW12.5, GSW13.5, GSW14.5, GSW15.5, GSW16.5, GSW21.5, GSW22.5, GSW23.5, GSW24.5, GSW9.5, IC10.1, IC11.1, IC12.1, IC13.1, IC14.1, IC15.1, IC16.1, IC21.1, IC22.1, IC23.1, IC24.1, IC9.1, ICAMP3.4, ICAMP4.4, ICAMP6.4
Routing:
- net GND: track 0.00 -> 607.2 mm, vias 0 -> 202
- net VCCA: track 0.00 -> 570.5 mm, vias 0 -> 1
- net +3V3: track 0.00 -> 463.8 mm, vias 0 -> 2
- net E_50SW6: track 0.00 -> 244.1 mm, vias 0 -> 6
- net L141_SCL: track 0.00 -> 220.4 mm, vias 0 -> 16
- net E_50SW1: track 0.00 -> 217.3 mm, vias 0 -> 7
- net E_50SW4: track 0.00 -> 216.9 mm, vias 0 -> 6
- net E_50SW8: track 0.00 -> 210.6 mm, vias 0 -> 5
- net E_50SW7: track 0.00 -> 205.6 mm, vias 0 -> 6
- net E_50SW2: track 0.00 -> 199.2 mm, vias 0 -> 7
- net E_50SW15: track 0.00 -> 198.4 mm, vias 0 -> 7
- net E_50SW14: track 0.00 -> 197.3 mm, vias 0 -> 6
- net L21_SDA: track 0.00 -> 192.8 mm, vias 0 -> 12
- net E_50SW13: track 0.00 -> 191.1 mm, vias 0 -> 9
- net N$59: track 0.00 -> 189.1 mm, vias 0 -> 4
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Other:
- board text added: "60"
- board text added: "62"
- board text added: "64"
- board text added: "65"
- board text added: "66"
- board text added: "69"
- board text added: "70"
- board text added: "74"
- board text added: "75"
- board text added: "76"
- board text added: "77"
- board text added: "78"
- board text added: "79"
- board text added: "81"
- board text added: "84"
- board text added: "85"
- board text added: "IN10"
- board text added: "IN11"
- board text added: "IN12"
- board text added: "IN13"
- board text added: "IN14"
- board text added: "IN15"
- board text added: "IN16"
- board text added: "IN5"
- board text added: "IN6"
- board text added: "IN7"
- board text added: "IN8"
- board text added: "IN9"
- board text removed: "10k"
- board text removed: "D0C .... D7C"
- board text removed: "D0D .... D7D"
- board text removed: "Reset"
