File: eagle/max10adc_v9.02_16chan.sch (EAGLE design)
At the start: 533 parts, among them IC1 MAX11115AUT+T, IC10 MAX11115AUT+T, IC11 MAX11115AUT+T, IC12 MAX11115AUT+T, IC13 MAX11115AUT+T, IC14 MAX11115AUT+T, IC15 MAX11115AUT+T, IC16 MAX11115AUT+T, IC2 MAX11115AUT+T, IC21 MAX11115AUT+T, IC22 MAX11115AUT+T, IC23 MAX11115AUT+T, IC24 MAX11115AUT+T, IC3 MAX11115AUT+T, IC4 MAX11115AUT+T, IC9 MAX11115AUT+T, K1 AQY21SOP, K10 AQY21SOP, K11 AQY21SOP, K12 AQY21SOP, K13 AQY21SOP, K14 AQY21SOP, K15 AQY21SOP, K16 AQY21SOP, K21 AQY21SOP, K22 AQY21SOP, K23 AQY21SOP, K24 AQY21SOP, K3 AQY21SOP, K5 AQY21SOP, K6 AQY21SOP, K9 AQY21SOP, U340G CH340G, X1 LTI-SASF54GT, X10 LTI-SASF54GT, X11 LTI-SASF54GT, X12 LTI-SASF54GT, X13 LTI-SASF54GT, X14 LTI-SASF54GT, X15 LTI-SASF54GT, X16 LTI-SASF54GT, X21 LTI-SASF54GT, X22 LTI-SASF54GT, X23 LTI-SASF54GT, X24 LTI-SASF54GT, X4 LTI-SASF54GT, X5 LTI-SASF54GT, X6 LTI-SASF54GT, X9 LTI-SASF54GT, Y1 ABL-12.000MHZ-B2

Commit message: with BOM
Parts:
- CGAIN1_1, CGAIN1_10, CGAIN1_11, CGAIN1_12, CGAIN1_13, CGAIN1_14, CGAIN1_15, CGAIN1_16, CGAIN1_21, CGAIN1_22, CGAIN1_23, CGAIN1_24, CGAIN1_3, CGAIN1_5, CGAIN1_6, CGAIN1_9: MPN 06033A330JAT2A -> (none)
- RG1_1, RG1_11, RG1_12, RG1_3, RG1_5, RG1_6, RG1_7, RG1_8, RG3_11, RG3_12, RG3_3, RG3_4, RG3_5, RG3_6, RG3_7, RG3_8: MPN MF-RES-0805-100k -> (none)
- RG2_1, RG2_11, RG2_12, RG2_3, RG2_5, RG2_6, RG2_7, RG2_8, RG4_11, RG4_12, RG4_3, RG4_4, RG4_5, RG4_6, RG4_7, RG4_8: MPN MF-RES-0805-1M -> (none)

Commit message: MAX11105
Parts:
- IC1, IC10, IC11, IC12, IC13, IC14, IC15, IC16, IC2, IC21, IC22, IC23, IC24, IC3, IC4, IC9: value MAX11115AUT+T -> MAX11105AUT+T; device SamacSys_Parts:MAX11115AUT+T -> SamacSys_Parts:MAX11105AUT+T
Changed lines of the file:
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@@
 <part name="+3V7" library="supply1" deviceset="+3V3" device=""/>
 <part name="ICAMP1" library="SamacSys_Parts" deviceset="OPA4322AIPWR" device=""/>
-<part name="IC4" library="SamacSys_Parts" deviceset="MAX11115AUT+T" device=""/>
+<part name="IC4" library="SamacSys_Parts" deviceset="MAX11105AUT+T" device=""/>
 <part name="X1" library="con-coax" library_urn="urn:adsk.eagle:library:133" deviceset="LTI-SASF54GT" device="" package3d_urn="urn:adsk.eagle:package:6232/1"/>
 <part name="IN1" library="Seeed-Connector" library_urn="urn:adsk.eagle:library:478" deviceset="DIP-BLACK-MALE-HEADER-VERT(2P-2.54)" device="" package3d_urn="urn:adsk.eagle:package:33132/1" value="2p-2.54"/>
@@
 </part>
 <part name="U$3" library="SparkFun-PowerSymbols" library_urn="urn:adsk.eagle:library:530" deviceset="VCCA" device=""/>
-<part name="IC1" library="SamacSys_Parts" deviceset="MAX11115AUT+T" device=""/>
+<part name="IC1" library="SamacSys_Parts" deviceset="MAX11105AUT+T" device=""/>
 <part name="GND11" library="supply1" deviceset="GND" device=""/>
 <part name="CADD3" library="rcl" deviceset="C-EU" device="C0805K" value="0.1uF">
@@
 </part>
 <part name="U$4" library="SparkFun-PowerSymbols" library_urn="urn:adsk.eagle:library:530" deviceset="VCCA" device=""/>
-<part name="IC2" library="SamacSys_Parts" deviceset="MAX11115AUT+T" device=""/>
+<part name="IC2" library="SamacSys_Parts" deviceset="MAX11105AUT+T" device=""/>
 <part name="GND17" library="supply1" deviceset="GND" device=""/>
 <part name="CADD4" library="rcl" deviceset="C-EU" device="C0805K" value="0.1uF">
@@
 </part>
 <part name="U$5" library="SparkFun-PowerSymbols" library_urn="urn:adsk.eagle:library:530" deviceset="VCCA" device=""/>
-<part name="IC3" library="SamacSys_Parts" deviceset="MAX11115AUT+T" device=""/>
+<part name="IC3" library="SamacSys_Parts" deviceset="MAX11105AUT+T" device=""/>
 <part name="IOEXPAND_0X22" library="microchip" deviceset="MCP23017" device="SS"/>
 <part name="+3V10" library="supply1" deviceset="+3V3" device=""/>
@@
 </part>
 <part name="ICAMP3" library="SamacSys_Parts" deviceset="OPA4322AIPWR" device=""/>
-<part name="IC9" library="SamacSys_Parts" deviceset="MAX11115AUT+T" device=""/>
+<part name="IC9" library="SamacSys_Parts" deviceset="MAX11105AUT+T" device=""/>
 <part name="ROFFSET10" library="resistor" library_urn="urn:adsk.eagle:library:348" deviceset="R-EU_" device="R0805" package3d_urn="urn:adsk.eagle:package:26059/1" value="200"/>
 <part name="ROFFSET11" library="resistor" library_urn="urn:adsk.eagle:library:348" deviceset="R-EU_" device="R0805" package3d_urn="urn:adsk.eagle:package:26059/1" value="200"/>
@@
 <attribute name="MPN" value="MF-CAP-0805-0.1uF"/>
 </part>
-<part name="IC10" library="SamacSys_Parts" deviceset="MAX11115AUT+T" device=""/>
+<part name="IC10" library="SamacSys_Parts" deviceset="MAX11105AUT+T" device=""/>
 <part name="CADD11" library="rcl" deviceset="C-EU" device="C0805K" value="0.1uF">
 <attribute name="MPN" value="MF-CAP-0805-0.1uF"/>
 </part>
-<part name="IC11" library="SamacSys_Parts" deviceset="MAX11115AUT+T" device=""/>
+<part name="IC11" library="SamacSys_Parts" deviceset="MAX11105AUT+T" device=""/>
 <part name="CADD12" library="rcl" deviceset="C-EU" device="C0805K" value="0.1uF">
 <attribute name="MPN" value="MF-CAP-0805-0.1uF"/>
 </part>
-<part name="IC12" library="SamacSys_Parts" deviceset="MAX11115AUT+T" device=""/>
+<part name="IC12" library="SamacSys_Parts" deviceset="MAX11105AUT+T" device=""/>
 <part name="GND93" library="supply1" deviceset="GND" device=""/>
 <part name="GSW9" library="74xx-little-us" deviceset="74*1G3157" device="DBVR">
@@
 </part>
 <part name="ICAMP4" library="SamacSys_Parts" deviceset="OPA4322AIPWR" device=""/>
-<part name="IC13" library="SamacSys_Parts" deviceset="MAX11115AUT+T" device=""/>
+<part name="IC13" library="SamacSys_Parts" deviceset="MAX11105AUT+T" device=""/>
 <part name="ROFFSET14" library="resistor" library_urn="urn:adsk.eagle:library:348" deviceset="R-EU_" device="R0805" package3d_urn="urn:adsk.eagle:package:26059/1" value="200"/>
 <part name="ROFFSET15" library="resistor" library_urn="urn:adsk.eagle:library:348" deviceset="R-EU_" device="R0805" package3d_urn="urn:adsk.eagle:package:26059/1" value="200"/>
@@
 <attribute name="MPN" value="MF-CAP-0805-0.1uF"/>
 </part>
-<part name="IC14" library="SamacSys_Parts" deviceset="MAX11115AUT+T" device=""/>
+<part name="IC14" library="SamacSys_Parts" deviceset="MAX11105AUT+T" device=""/>
 <part name="CADD15" library="rcl" deviceset="C-EU" device="C0805K" value="0.1uF">
 <attribute name="MPN" value="MF-CAP-0805-0.1uF"/>
 </part>
-<part name="IC15" library="SamacSys_Parts" deviceset="MAX11115AUT+T" device=""/>
+<part name="IC15" library="SamacSys_Parts" deviceset="MAX11105AUT+T" device=""/>
 <part name="CADD16" library="rcl" deviceset="C-EU" device="C0805K" value="0.1uF">
 <attribute name="MPN" value="MF-CAP-0805-0.1uF"/>
 </part>
-<part name="IC16" library="SamacSys_Parts" deviceset="MAX11115AUT+T" device=""/>
+<part name="IC16" library="SamacSys_Parts" deviceset="MAX11105AUT+T" device=""/>
 <part name="C5VOPAMP6" library="rcl" deviceset="C-EU" device="C0805K" value="0.1uF">
 <attribute name="MPN" value="MF-CAP-0805-0.1uF"/>
@@
 </part>
 <part name="ICAMP6" library="SamacSys_Parts" deviceset="OPA4322AIPWR" device=""/>
-<part name="IC21" library="SamacSys_Parts" deviceset="MAX11115AUT+T" device=""/>
+<part name="IC21" library="SamacSys_Parts" deviceset="MAX11105AUT+T" device=""/>
 <part name="ROFFSET22" library="resistor" library_urn="urn:adsk.eagle:library:348" deviceset="R-EU_" device="R0805" package3d_urn="urn:adsk.eagle:package:26059/1" value="200"/>
 <part name="ROFFSET23" library="resistor" library_urn="urn:adsk.eagle:library:348" deviceset="R-EU_" device="R0805" package3d_urn="urn:adsk.eagle:package:26059/1" value="200"/>
@@
 <attribute name="MPN" value="MF-CAP-0805-0.1uF"/>
 </part>
-<part name="IC22" library="SamacSys_Parts" deviceset="MAX11115AUT+T" device=""/>
+<part name="IC22" library="SamacSys_Parts" deviceset="MAX11105AUT+T" device=""/>
 <part name="CADD23" library="rcl" deviceset="C-EU" device="C0805K" value="0.1uF">
 <attribute name="MPN" value="MF-CAP-0805-0.1uF"/>
 </part>
-<part name="IC23" library="SamacSys_Parts" deviceset="MAX11115AUT+T" device=""/>
+<part name="IC23" library="SamacSys_Parts" deviceset="MAX11105AUT+T" device=""/>
 <part name="CADD24" library="rcl" deviceset="C-EU" device="C0805K" value="0.1uF">
 <attribute name="MPN" value="MF-CAP-0805-0.1uF"/>
 </part>
-<part name="IC24" library="SamacSys_Parts" deviceset="MAX11115AUT+T" device=""/>
+<part name="IC24" library="SamacSys_Parts" deviceset="MAX11105AUT+T" device=""/>
 <part name="GND117" library="supply1" deviceset="GND" device=""/>
 <part name="GSW13" library="74xx-little-us" deviceset="74*1G3157" device="DBVR">
@@
 <attribute name="VALUE" x="60.96" y="58.42" size="1.778" layer="96"/>
 </instance>
-<instance part="GOLD_ORB_SM1" gate="G$1" x="15.24" y="38.1" smashed="yes"/>
+<instance part="GOLD_ORB_SM1" gate="G$1" x="15.24" y="33.02" smashed="yes"/>
 <instance part="IC4" gate="G$1" x="38.1" y="165.1" smashed="yes">
 <attribute name="NAME" x="44.45" y="172.72" size="1.778" layer="95" align="center-left"/>

Commit message: with 24pF fixed caps
Parts:
- removed CH1, CH10, CH11, CH12, CH13, CH14, CH15, CH16, CH2, CH3, CH4, CH5, CH6, CH7, CH8, CH9, CL1, CL10, CL11, CL12, CL13, CL14, CL15, CL16, CL2, CL3, CL4, CL5, CL6, CL7, CL8, CL9: 8-45pF, SparkFun-Passives:CAP_ADJSMD
- added CGN1, CGN10, CGN11, CGN12, CGN13, CGN14, CGN15, CGN16, CGN17, CGN18, CGN19, CGN2, CGN20, CGN21, CGN22, CGN23, CGN24, CGN25, CGN26, CGN27, CGN28, CGN29, CGN3, CGN30, CGN31, CGN32, CGN4, CGN5, CGN6, CGN7, CGN8, CGN9: 24pF, rcl@1:C-USC0603
Connections:
- net CGAIN1: now also CGN1.2; no longer CL1.4
- net CGAIN10: now also CGN8.2; no longer CH3.4
- net CGAIN11: now also CGN6.1; no longer CL4.4
- net CGAIN12: now also CGN7.2; no longer CH4.4
- net CGAIN17: now also CGN10.2; no longer CL5.4
- net CGAIN18: now also CGN9.2; no longer CH5.4
- net CGAIN19: now also CGN22.2; no longer CL6.4
- net CGAIN2: now also CGN2.2; no longer CH1.4
- net CGAIN20: now also CGN21.2; no longer CH6.4
- net CGAIN21: now also CGN11.1; no longer CL7.4
- net CGAIN22: now also CGN12.1; no longer CH7.4
- net CGAIN23: now also CGN23.1; no longer CL8.4
- net CGAIN24: now also CGN24.1; no longer CH8.4
- net CGAIN25: now also CGN14.2; no longer CL9.4
- net CGAIN26: now also CGN13.2; no longer CH9.4
- net CGAIN27: now also CGN26.2; no longer CL10.4
- net CGAIN28: now also CGN25.2; no longer CH10.4
- net CGAIN29: now also CGN15.1; no longer CL11.4
- net CGAIN30: now also CGN16.1; no longer CH11.4
- net CGAIN31: now also CGN27.1; no longer CL12.4
- net CGAIN32: now also CGN28.1; no longer CH12.4
- net CGAIN41: now also CGN18.2; no longer CL13.4
- net CGAIN42: now also CGN17.2; no longer CH13.4
- net CGAIN43: now also CGN30.2; no longer CL14.4
- net CGAIN44: now also CGN29.2; no longer CH14.4
- net CGAIN45: now also CGN19.1; no longer CL15.4
- net CGAIN46: now also CGN20.1; no longer CH15.4
- net CGAIN47: now also CGN31.1; no longer CL16.4
- net CGAIN48: now also CGN32.1; no longer CH16.4
- net CGAIN5: now also CGN4.2; no longer CL2.4
- net CGAIN6: now also CGN3.2; no longer CH2.4
- net CGAIN9: now also CGN5.1; no longer CL3.4
- net INAMINUS1: now also CGN1.1, CGN2.1; no longer CH1.3, CL1.3
- net INAMINUS10: now also CGN25.1, CGN26.1; no longer CH10.3, CL10.3
- net INAMINUS11: now also CGN15.2, CGN16.2; no longer CH11.3, CL11.3
- net INAMINUS12: now also CGN27.2, CGN28.2; no longer CH12.3, CL12.3
- net INAMINUS13: now also CGN17.1, CGN18.1; no longer CH13.3, CL13.3
- net INAMINUS14: now also CGN29.1, CGN30.1; no longer CH14.3, CL14.3
- net INAMINUS15: now also CGN19.2, CGN20.2; no longer CH15.3, CL15.3
- net INAMINUS16: now also CGN31.2, CGN32.2; no longer CH16.3, CL16.3
- net INAMINUS2: now also CGN3.1, CGN4.1; no longer CH2.3, CL2.3
- net INAMINUS3: now also CGN5.2, CGN8.1; no longer CH3.3, CL3.3
- net INAMINUS4: now also CGN6.2, CGN7.1; no longer CH4.3, CL4.3
- net INAMINUS5: now also CGN10.1, CGN9.1; no longer CH5.3, CL5.3
- net INAMINUS6: now also CGN21.1, CGN22.1; no longer CH6.3, CL6.3
- net INAMINUS7: now also CGN11.2, CGN12.2; no longer CH7.3, CL7.3
- net INAMINUS8: now also CGN23.2, CGN24.2; no longer CH8.3, CL8.3
- net INAMINUS9: now also CGN13.1, CGN14.1; no longer CH9.3, CL9.3
Other:
- moved on the sheet: CGAIN1_10, CGAIN1_11, CGAIN1_12, CGAIN1_14, CGAIN1_15, CGAIN1_16, CGAIN1_22, CGAIN1_23, CGAIN1_24, CGAIN1_3, CGAIN1_5, CGAIN1_6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

Commit message: test3
Connections:
- net N$48 renamed 5VC3
- net N$49 renamed 5VC5
Changed lines of the file:
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@@
 <class number="1" name="gnd" width="0.3048" drill="0">
 </class>
-<class number="2" name="three" width="0.1524" drill="0">
+<class number="2" name="three" width="0.3048" drill="0">
 </class>
 <class number="3" name="five" width="0.381" drill="0">
@@
 </segment>
 </net>
-<net name="N$49" class="3">
+<net name="5VC5" class="3">
 <segment>
 <pinref part="L1" gate="G$1" pin="2"/>
@@
 </segment>
 </net>
-<net name="N$48" class="3">
+<net name="5VC3" class="3">
 <segment>
 <pinref part="L2" gate="G$1" pin="2"/>

Commit message: front panel with 50 Ohm termination and SMAs
Parts:
- removed BJ1, BJ2, BJ3, BJ4: 6p-2.54, Seeed-Connector:DIP-BLACK-MALE-HEADER(6P-2.54)
- removed IN1, IN10, IN11, IN12, IN13, IN14, IN15, IN16, IN2, IN3, IN4, IN5, IN6, IN7, IN8, IN9: 2p-2.54, Seeed-Connector:DIP-BLACK-MALE-HEADER-VERT(2P-2.54)
- removed R50-1, R50-10, R50-11, R50-12, R50-17, R50-18, R50-19, R50-2, R50-20, R50-21, R50-22, R50-23, R50-24, R50-3, R50-33, R50-34, R50-35, R50-36, R50-37, R50-38, R50-39, R50-4, R50-40, R50-41, R50-42, R50-43, R50-44, R50-45, R50-46, R50-47, R50-48, R50-49, R50-50, R50-51, R50-52, R50-53, R50-54, R50-55, R50-56, R50-57, R50-58, R50-59, R50-60, R50-61, R50-62, R50-63, R50-64, R50-81, R50-82, R50-83, R50-84, R50-85, R50-86, R50-87, R50-88, R50-89, R50-9, R50-90, R50-91, R50-92, R50-93, R50-94, R50-95, R50-96: 200R, resistor:R-EU_R0805
- removed S1, S10, S12, S18, S20, S22, S24, S26, S28, S30, S32, S42, S44, S46, S48, S5: JS202011SCQN, switch-ck:JS202011SCQN
- removed X1, X10, X11, X12, X13, X14, X15, X16, X21, X22, X23, X24, X4, X5, X6, X9: LTI-SASF54GT, con-coax:LTI-SASF54GT
- added H1, H2, H3, H4, H5, H6: STANDOFF_ELECTRICAL, SparkFun-Hardware:STANDOFF_ELECTRICAL
- added JP2: (no value), pinhead:PINHD-2X20/90
- added JP3: (no value), pinhead:PINHD-2X20
Connections:
- removed net N50_1: R50-1.1, R50-2.1, R50-3.1, R50-4.1, S1.3
- removed net N50_10: R50-53.1, R50-54.1, R50-55.1, R50-56.1, S28.3
- removed net N50_11: R50-57.1, R50-58.1, R50-59.1, R50-60.1, S30.3
- removed net N50_12: R50-61.1, R50-62.1, R50-63.1, R50-64.1, S32.3
- removed net N50_13: R50-81.1, R50-82.1, R50-83.1, R50-84.1, S42.3
- removed net N50_14: R50-85.1, R50-86.1, R50-87.1, R50-88.1, S44.3
- removed net N50_15: R50-89.1, R50-90.1, R50-91.1, R50-92.1, S46.3
- removed net N50_16: R50-93.1, R50-94.1, R50-95.1, R50-96.1, S48.3
- removed net N50_2: R50-10.1, R50-11.1, R50-12.1, R50-9.1, S5.3
- removed net N50_3: R50-17.1, R50-18.1, R50-19.1, R50-20.1, S10.3
- removed net N50_4: R50-21.1, R50-22.1, R50-23.1, R50-24.1, S12.3
- removed net N50_5: R50-33.1, R50-34.1, R50-35.1, R50-36.1, S18.3
- removed net N50_6: R50-37.1, R50-38.1, R50-39.1, R50-40.1, S20.3
- removed net N50_7: R50-41.1, R50-42.1, R50-43.1, R50-44.1, S22.3
- removed net N50_8: R50-45.1, R50-46.1, R50-47.1, R50-48.1, S24.3
- removed net N50_9: R50-49.1, R50-50.1, R50-51.1, R50-52.1, S26.3
- net AIN1: now also JP2.6, JP3.6
- net E_50SW1: now also JP2.37, JP3.37; no longer S1.5
- net E_50SW10: now also JP2.19, JP3.19; no longer S28.5
- net E_50SW11: now also JP2.17, JP3.17; no longer S30.5
- net E_50SW12: now also JP2.15, JP3.15; no longer S32.5
- net E_50SW13: now also JP2.13, JP3.13; no longer S42.5
- net E_50SW14: now also JP2.11, JP3.11; no longer S44.5
- net E_50SW15: now also JP2.9, JP3.9; no longer S46.5
- net E_50SW16: now also JP2.7, JP3.7; no longer S48.5
- net E_50SW2: now also JP2.35, JP3.35; no longer S5.5
- net E_50SW3: now also JP2.33, JP3.33; no longer S10.5
- net E_50SW4: now also JP2.31, JP3.31; no longer S12.5
- net E_50SW5: now also JP2.29, JP3.29; no longer S18.5
- net E_50SW6: now also JP2.27, JP3.27; no longer S20.5
- net E_50SW7: now also JP2.25, JP3.25; no longer S22.5
- net E_50SW8: now also JP2.23, JP3.23; no longer S24.5
- net E_50SW9: now also JP2.21, JP3.21; no longer S26.5
- net GND: now also H1.P$1, H2.P$1, H3.P$1, H4.P$1, H5.P$1, H6.P$1, JP2.2, JP2.40, JP3.2, JP3.40; no longer BJ1.1, BJ2.1, BJ3.1, BJ4.1, IN1.1, IN10.1, IN11.1, IN12.1, IN13.1, IN14.1, IN15.1, IN16.1, IN2.1, IN3.1, IN4.1, IN5.1, IN6.1, IN7.1, IN8.1, IN9.1, R50-1.2, R50-10.2, R50-11.2, R50-12.2, R50-17.2, R50-18.2, R50-19.2, R50-2.2, R50-20.2, R50-21.2, R50-22.2, R50-23.2, R50-24.2, R50-3.2, R50-33.2, R50-34.2, R50-35.2, R50-36.2, R50-37.2, R50-38.2, R50-39.2, R50-4.2, R50-40.2, R50-41.2, R50-42.2, R50-43.2, R50-44.2, R50-45.2, R50-46.2, R50-47.2, R50-48.2, R50-49.2, R50-50.2, R50-51.2, R50-52.2, R50-53.2, R50-54.2, R50-55.2, R50-56.2, R50-57.2, R50-58.2, R50-59.2, R50-60.2, R50-61.2, R50-62.2, R50-63.2, R50-64.2, R50-81.2, R50-82.2, R50-83.2, R50-84.2, R50-85.2, R50-86.2, R50-87.2, R50-88.2, R50-89.2, R50-9.2, R50-90.2, R50-91.2, R50-92.2, R50-93.2, R50-94.2, R50-95.2, R50-96.2, S1.6, S10.6, S12.6, S18.6, S20.6, S22.6, S24.6, S26.6, S28.6, S30.6, S32.6, S42.6, S44.6, S46.6, S48.6, S5.6, X1.2, X10.2, X11.2, X12.2, X13.2, X14.2, X15.2, X16.2, X21.2, X22.2, X23.2, X24.2, X4.2, X5.2, X6.2, X9.2
- net INJ1: now also JP2.38, JP3.38; no longer BJ1.5, IN1.2, S1.2, X1.1
- net INJ10: now also JP2.20, JP3.20; no longer BJ3.4, IN10.2, S28.2, X14.1
- net INJ11: now also JP2.18, JP3.18; no longer BJ3.3, IN11.2, S30.2, X15.1
- net INJ12: now also JP2.16, JP3.16; no longer BJ3.2, IN12.2, S32.2, X16.1
- net INJ13: now also JP2.14, JP3.14; no longer BJ4.5, IN13.2, S42.2, X21.1
- net INJ14: now also JP2.12, JP3.12; no longer BJ4.4, IN14.2, S44.2, X22.1
- net INJ15: now also JP2.10, JP3.10; no longer BJ4.3, IN15.2, S46.2, X23.1
- net INJ16: now also JP2.8, JP3.8; no longer BJ4.2, IN16.2, S48.2, X24.1
- net INJ2: now also JP2.36, JP3.36; no longer BJ1.4, IN2.2, S5.2, X5.1
- net INJ3: now also JP2.34, JP3.34; no longer BJ1.3, IN3.2, S10.2, X4.1
- net INJ4: now also JP2.32, JP3.32; no longer BJ1.2, IN4.2, S12.2, X6.1
- net INJ5: now also JP2.30, JP3.30; no longer BJ2.5, IN5.2, S18.2, X9.1
- net INJ6: now also JP2.28, JP3.28; no longer BJ2.4, IN6.2, S20.2, X10.1
- net INJ7: now also JP2.26, JP3.26; no longer BJ2.3, IN7.2, S22.2, X11.1
- net INJ8: now also JP2.24, JP3.24; no longer BJ2.2, IN8.2, S24.2, X12.1
- net INJ9: now also JP2.22, JP3.22; no longer BJ3.5, IN9.2, S26.2, X13.1
- net IO_100: now also JP2.5, JP3.5
- net IO_101: now also JP2.3, JP3.3
- net L121: now also JP2.4, JP3.4
- net VCCA: now also JP2.1, JP2.39, JP3.1, JP3.39; no longer BJ1.6, BJ2.6, BJ3.6, BJ4.6
Other:
- note added: "IO connectors"
- note removed: "4 200 Ohm resistors in parallel for 50 Ohm termination"
- note removed: "Switch for 1M / 50 Ohm input impedance"

Commit message: back connectors
Parts:
- removed PIN_AIN_IO2_PWRGND, PIN_ANALOG_IOEXP, PIN_DIGITAL_1: 15-91-2160, pinhead+:PINHD-2X8SMT
- added JP4: (no value), pinhead:PINHD-2X20/90
Connections:
- net +3V3: now also JP4.38; no longer PIN_AIN_IO2_PWRGND.14, PIN_AIN_IO2_PWRGND.16, PIN_AIN_IO2_PWRGND.3, PIN_ANALOG_IOEXP.15
- net +5V: no longer PIN_AIN_IO2_PWRGND.10, PIN_AIN_IO2_PWRGND.12
- net A10: now also JP4.23; no longer PIN_ANALOG_IOEXP.8
- net A11: now also JP4.18; no longer PIN_ANALOG_IOEXP.10
- net A12: now also JP4.20; no longer PIN_ANALOG_IOEXP.12
- net A13: now also JP4.22; no longer PIN_ANALOG_IOEXP.14
- net A14: now also JP4.24; no longer PIN_ANALOG_IOEXP.16
- net A6: now also JP4.17; no longer PIN_ANALOG_IOEXP.2
- net A7: now also JP4.19; no longer PIN_ANALOG_IOEXP.4
- net A8: now also JP4.21; no longer PIN_ANALOG_IOEXP.6
- net AIN1: now also JP4.39; no longer PIN_AIN_IO2_PWRGND.2
- net D0C: now also JP4.1; no longer PIN_DIGITAL_1.1
- net D0D: now also JP4.2; no longer PIN_DIGITAL_1.2
- net D1C: now also JP4.3; no longer PIN_DIGITAL_1.3
- net D1D: now also JP4.4; no longer PIN_DIGITAL_1.4
- net D2C: now also JP4.5; no longer PIN_DIGITAL_1.5
- net D2D: now also JP4.6; no longer PIN_DIGITAL_1.6
- net D3C: now also JP4.7; no longer PIN_DIGITAL_1.7
- net D3D: now also JP4.8; no longer PIN_DIGITAL_1.8
- net D4C: now also JP4.9; no longer PIN_DIGITAL_1.9
- net D4D: now also JP4.10; no longer PIN_DIGITAL_1.10
- net D5C: now also JP4.11; no longer PIN_DIGITAL_1.11
- net D5D: now also JP4.12; no longer PIN_DIGITAL_1.12
- net D6C: now also JP4.13; no longer PIN_DIGITAL_1.13
- net D6D: now also JP4.14; no longer PIN_DIGITAL_1.14
- net D7C: now also JP4.15; no longer PIN_DIGITAL_1.15
- net D7D: now also JP4.16; no longer PIN_DIGITAL_1.16
- net GND: now also JP4.40; no longer PIN_AIN_IO2_PWRGND.1, PIN_AIN_IO2_PWRGND.6, PIN_AIN_IO2_PWRGND.8, PIN_ANALOG_IOEXP.9
- net IO_100: now also JP4.33; no longer PIN_AIN_IO2_PWRGND.13
- net IO_101: now also JP4.35; no longer PIN_AIN_IO2_PWRGND.15
- net IO_CLK_88: now also JP4.25; no longer PIN_AIN_IO2_PWRGND.5
- net IO_CLK_89: now also JP4.27; no longer PIN_AIN_IO2_PWRGND.7
- net IO_CLK_90: now also JP4.29; no longer PIN_AIN_IO2_PWRGND.9
- net IO_CLK_91: now also JP4.31; no longer PIN_AIN_IO2_PWRGND.11
- net L120_LED1: now also JP4.36; no longer PIN_ANALOG_IOEXP.1
- net L121: now also JP4.37; no longer PIN_AIN_IO2_PWRGND.4
- net L141_SCL: now also JP4.28; no longer PIN_ANALOG_IOEXP.11
- net L21_SDA: now also JP4.26; no longer PIN_ANALOG_IOEXP.13
- net L22_LED2: now also JP4.34; no longer PIN_ANALOG_IOEXP.3
- net L24_LED3: now also JP4.32; no longer PIN_ANALOG_IOEXP.5
- net L25_LED4: now also JP4.30; no longer PIN_ANALOG_IOEXP.7
Other:
- moved on the sheet: PIN_RIGHT
