File: eagle/max10adc_v9.02_16chan_frontpanel.sch (EAGLE design)
At the start: 106 parts, among them CN1 8p-2.54, X1 BU-SMA-V, X10 BU-SMA-V, X11 BU-SMA-V, X12 BU-SMA-V, X13 BU-SMA-V, X14 BU-SMA-V, X15 BU-SMA-V, X16 BU-SMA-V, X2 BU-SMA-V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

Commit message: back connectors
Parts:
- removed CN1: 8p-2.54, Seeed-Connector:DIP-BLACK-FEMALE-HEADER-VERT(8P-2.54)
- removed H1: STANDOFF_ELECTRICAL, SparkFun-Hardware:STANDOFF_ELECTRICAL
- added J1, J2: 4p-2.54, Seeed-Connector:DIP-BLACK-MALE-HEADER-VERT(4P-2.54)
Connections:
- net AIN1: now also J2.P$3; no longer CN1.3
- net GND: now also J2.P$1, J2.P$2; no longer CN1.1, CN1.2, H1.P$1
- net IO_100: now also J1.P$2; no longer CN1.6
- net IO_101: now also J1.P$1; no longer CN1.5
- net L121: now also J2.P$4; no longer CN1.4
- net VCCA: now also J1.P$3, J1.P$4; no longer CN1.7, CN1.8
Changed lines of the file:
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@@
 <parts>
 <part name="FRAME2" library="frames" library_urn="urn:adsk.eagle:library:229" deviceset="A3L-LOC" device=""/>
-<part name="H1" library="SparkFun-Hardware" deviceset="STANDOFF_ELECTRICAL" device="" package3d_urn="urn:adsk.eagle:package:38631/1"/>
 <part name="H2" library="SparkFun-Hardware" deviceset="STANDOFF_ELECTRICAL" device="" package3d_urn="urn:adsk.eagle:package:38631/1"/>
 <part name="JP3" library="pinhead" library_urn="urn:adsk.eagle:library:325" deviceset="PINHD-2X20" device="" package3d_urn="urn:adsk.eagle:package:22443/2"/>
-<part name="GND9" library="supply1" deviceset="GND" device=""/>
 <part name="GND27" library="supply1" deviceset="GND" device=""/>
 <part name="GND1" library="supply1" deviceset="GND" device=""/>
@@
 <part name="GND11" library="supply1" deviceset="GND" device=""/>
 <part name="GND21" library="supply1" deviceset="GND" device=""/>
-<part name="CN1" library="Seeed-Connector" library_urn="urn:adsk.eagle:library:478" deviceset="DIP-BLACK-FEMALE-HEADER-VERT(8P-2.54)" device="" package3d_urn="urn:adsk.eagle:package:33113/1" value="8p-2.54"/>
 <part name="GND22" library="supply1" deviceset="GND" device=""/>
+<part name="J1" library="Seeed-Connector" library_urn="urn:adsk.eagle:library:478" deviceset="DIP-BLACK-MALE-HEADER-VERT(4P-2.54)" device="" package3d_urn="urn:adsk.eagle:package:33137/1" value="4p-2.54"/>
+<part name="J2" library="Seeed-Connector" library_urn="urn:adsk.eagle:library:478" deviceset="DIP-BLACK-MALE-HEADER-VERT(4P-2.54)" device="" package3d_urn="urn:adsk.eagle:package:33137/1" value="4p-2.54"/>
 </parts>
 <sheets>
@@
 <attribute name="VALUE" x="285.75" y="55.88" size="1.778" layer="96"/>
 </instance>
-<instance part="H1" gate="G$1" x="20.32" y="246.38" smashed="yes">
-<attribute name="NAME" x="20.32" y="251.714" size="1.27" layer="95" font="vector" align="bottom-center"/>
-<attribute name="VALUE" x="20.32" y="241.046" size="1.27" layer="96" font="vector" rot="R180" align="bottom-center"/>
-</instance>
 <instance part="H2" gate="G$1" x="363.22" y="243.84" smashed="yes">
 <attribute name="NAME" x="363.22" y="249.174" size="1.27" layer="95" font="vector" align="bottom-center"/>
 <attribute name="VALUE" x="363.22" y="238.506" size="1.27" layer="96" font="vector" rot="R180" align="bottom-center"/>
 </instance>
-<instance part="GND9" gate="1" x="27.94" y="236.22" smashed="yes">
-<attribute name="VALUE" x="25.4" y="233.68" size="1.778" layer="96"/>
-</instance>
 <instance part="GND27" gate="1" x="370.84" y="233.68" smashed="yes">
 <attribute name="VALUE" x="368.3" y="231.14" size="1.778" layer="96"/>
@@
 <attribute name="VALUE" x="142.24" y="137.16" size="1.778" layer="96" rot="MR0"/>
 </instance>
-<instance part="CN1" gate="G$1" x="86.36" y="106.68" smashed="yes" rot="R270">
-<attribute name="NAME" x="97.79" y="114.3" size="1.27" layer="95" ratio="10" rot="R270"/>
-<attribute name="VALUE" x="97.79" y="106.68" size="1.27" layer="96" ratio="10" rot="R270"/>
-</instance>
 <instance part="GND22" gate="1" x="106.68" y="106.68" smashed="yes" rot="MR0">
 <attribute name="VALUE" x="109.22" y="104.14" size="1.778" layer="96" rot="MR0"/>
+</instance>
+<instance part="J1" gate="G$1" x="81.28" y="96.52" smashed="yes" rot="R270">
+<attribute name="NAME" x="87.63" y="104.14" size="1.27" layer="95" ratio="10" rot="R270"/>
+<attribute name="VALUE" x="87.63" y="97.79" size="1.27" layer="96" ratio="10" rot="R270"/>
+</instance>
+<instance part="J2" gate="G$1" x="91.44" y="106.68" smashed="yes" rot="R270">
+<attribute name="NAME" x="97.79" y="114.3" size="1.27" layer="95" ratio="10" rot="R270"/>
+<attribute name="VALUE" x="97.79" y="107.95" size="1.27" layer="96" ratio="10" rot="R270"/>
 </instance>
 </instances>
@@
 <wire x1="297.18" y1="109.22" x2="314.96" y2="109.22" width="0.1524" layer="91"/>
 <label x="307.34" y="109.22" size="1.778" layer="95"/>
-</segment>
-<segment>
-<pinref part="H1" gate="G$1" pin="P$1"/>
-<wire x1="27.94" y1="246.38" x2="27.94" y2="238.76" width="0.1524" layer="91"/>
-<pinref part="GND9" gate="1" pin="GND"/>
 </segment>
 <segment>
@@
 </segment>
 <segment>
-<pinref part="CN1" gate="G$1" pin="1"/>
 <wire x1="106.68" y1="109.22" x2="106.68" y2="114.3" width="0.1524" layer="91"/>
+<pinref part="GND22" gate="1" pin="GND"/>
 <wire x1="106.68" y1="114.3" x2="95.25" y2="114.3" width="0.1524" layer="91"/>
-<pinref part="CN1" gate="G$1" pin="2"/>
+<pinref part="J2" gate="G$1" pin="P$1"/>
+<pinref part="J2" gate="G$1" pin="P$2"/>
 <wire x1="92.71" y1="114.3" x2="95.25" y2="114.3" width="0.1524" layer="91"/>
 <junction x="95.25" y="114.3"/>
-<pinref part="GND22" gate="1" pin="GND"/>
 </segment>
 </net>
@@
 </segment>
 <segment>
-<pinref part="CN1" gate="G$1" pin="8"/>
-<wire x1="77.47" y1="114.3" x2="68.58" y2="114.3" width="0.1524" layer="91"/>
-<pinref part="CN1" gate="G$1" pin="7"/>
-<wire x1="80.01" y1="114.3" x2="77.47" y2="114.3" width="0.1524" layer="91"/>
-<junction x="77.47" y="114.3"/>
-<label x="68.58" y="114.3" size="1.778" layer="95"/>
+<label x="76.2" y="106.68" size="1.778" layer="95" rot="R90"/>
+<wire x1="77.47" y1="104.14" x2="77.47" y2="109.474" width="0.1524" layer="91"/>
+<pinref part="J1" gate="G$1" pin="P$4"/>
+<pinref part="J1" gate="G$1" pin="P$3"/>
+<wire x1="77.47" y1="104.14" x2="77.3938" y2="104.14" width="0.1524" layer="91"/>
+<wire x1="80.01" y1="104.14" x2="77.47" y2="104.14" width="0.1524" layer="91"/>
+<junction x="77.47" y="104.14"/>
 </segment>
 </net>
@@
 <wire x1="60.96" y1="147.32" x2="85.09" y2="147.32" width="0.1524" layer="91"/>
 <label x="66.04" y="147.32" size="1.778" layer="95"/>
-<pinref part="CN1" gate="G$1" pin="5"/>
-<wire x1="85.09" y1="147.32" x2="85.09" y2="114.3" width="0.1524" layer="91"/>
+<wire x1="85.09" y1="147.32" x2="85.09" y2="104.14" width="0.1524" layer="91"/>
+<pinref part="J1" gate="G$1" pin="P$1"/>
 </segment>
 </net>
@@
 <wire x1="22.86" y1="147.32" x2="38.1" y2="147.32" width="0.1524" layer="91"/>
 <label x="27.94" y="147.32" size="1.778" layer="95"/>
-<pinref part="CN1" gate="G$1" pin="6"/>
-<wire x1="82.55" y1="114.3" x2="82.55" y2="121.92" width="0.1524" layer="91"/>
+<wire x1="82.55" y1="104.14" x2="82.55" y2="121.92" width="0.1524" layer="91"/>
 <wire x1="82.55" y1="121.92" x2="38.1" y2="121.92" width="0.1524" layer="91"/>
 <wire x1="38.1" y1="121.92" x2="38.1" y2="147.32" width="0.1524" layer="91"/>
+<pinref part="J1" gate="G$1" pin="P$2"/>
 </segment>
 </net>
@@
 <wire x1="116.84" y1="147.32" x2="116.84" y2="119.38" width="0.1524" layer="91"/>
 <wire x1="116.84" y1="119.38" x2="87.63" y2="119.38" width="0.1524" layer="91"/>
-<pinref part="CN1" gate="G$1" pin="4"/>
 <wire x1="87.63" y1="119.38" x2="87.63" y2="114.3" width="0.1524" layer="91"/>
+<pinref part="J2" gate="G$1" pin="P$4"/>
 </segment>
 </net>
@@
 <wire x1="139.7" y1="147.32" x2="152.4" y2="147.32" width="0.1524" layer="91"/>
 <label x="144.78" y="147.32" size="1.778" layer="95"/>
-<pinref part="CN1" gate="G$1" pin="3"/>
 <wire x1="90.17" y1="114.3" x2="90.17" y2="116.84" width="0.1524" layer="91"/>
 <wire x1="90.17" y1="116.84" x2="152.4" y2="116.84" width="0.1524" layer="91"/>
 <wire x1="152.4" y1="116.84" x2="152.4" y2="147.32" width="0.1524" layer="91"/>
-</segment>
-</net>
+<pinref part="J2" gate="G$1" pin="P$3"/>
+</segment>
+</net>
