File: eagle/rack_backplane_v9.0.sch (EAGLE design)
At the start: 2 parts

Commit message: before routing
Parts:
- removed PIN_AIN_IO2_PWRGND, PIN_ANALOG_IOEXP1: 15-91-2160, pinhead:PINHD-2X8/90
- added PIN_AIN_PWRGND1, PIN_AIN_PWRGND10, PIN_AIN_PWRGND11, PIN_AIN_PWRGND12, PIN_AIN_PWRGND13, PIN_AIN_PWRGND14, PIN_AIN_PWRGND15, PIN_AIN_PWRGND16, PIN_AIN_PWRGND17, PIN_AIN_PWRGND18, PIN_AIN_PWRGND19, PIN_AIN_PWRGND2, PIN_AIN_PWRGND20, PIN_AIN_PWRGND21, PIN_AIN_PWRGND3, PIN_AIN_PWRGND4, PIN_AIN_PWRGND5, PIN_AIN_PWRGND6, PIN_AIN_PWRGND7, PIN_AIN_PWRGND8, PIN_AIN_PWRGND9, PIN_ANALOG_1, PIN_ANALOG_10, PIN_ANALOG_11, PIN_ANALOG_12, PIN_ANALOG_13, PIN_ANALOG_14, PIN_ANALOG_15, PIN_ANALOG_16, PIN_ANALOG_17, PIN_ANALOG_18, PIN_ANALOG_19, PIN_ANALOG_2, PIN_ANALOG_20, PIN_ANALOG_21, PIN_ANALOG_3, PIN_ANALOG_4, PIN_ANALOG_5, PIN_ANALOG_6, PIN_ANALOG_7, PIN_ANALOG_8, PIN_ANALOG_9: 15-91-2160, pinhead:PINHD-2X8
Connections:
- removed net +3V3: PIN_AIN_IO2_PWRGND.3
- removed net CLKOUTTOLEFT_29: PIN_ANALOG_IOEXP1.2
- removed net IO_100: PIN_AIN_IO2_PWRGND.13
- removed net IO_101: PIN_AIN_IO2_PWRGND.15
- removed net IO_CLK_88: PIN_AIN_IO2_PWRGND.5
- removed net IO_CLK_89: PIN_AIN_IO2_PWRGND.7
- removed net IO_CLK_90: PIN_AIN_IO2_PWRGND.9
- removed net IO_CLK_91: PIN_AIN_IO2_PWRGND.11
- removed net SERIALFROMLEFT_98: PIN_ANALOG_IOEXP1.14
- removed net SERIALTOLEFT_96: PIN_ANALOG_IOEXP1.12
- removed net SPARELEFT_102: PIN_ANALOG_IOEXP1.4
- removed net TRIGINFROMLEFT_28: PIN_ANALOG_IOEXP1.8
- removed net TRIGOUTTOLEFT_106: PIN_ANALOG_IOEXP1.10
- new net 3V3_1: PIN_AIN_PWRGND1.3
- new net 3V3_2: PIN_AIN_PWRGND2.3
- new net AIN1_2: PIN_AIN_PWRGND2.2
- new net IO_100_1: PIN_AIN_PWRGND1.13
- new net IO_100_2: PIN_AIN_PWRGND2.13
- new net IO_101_1: PIN_AIN_PWRGND1.15, PIN_ANALOG_21.4
- new net IO_101_10: PIN_AIN_PWRGND10.15, PIN_AIN_PWRGND21.7
- new net IO_101_11: PIN_AIN_PWRGND11.15, PIN_AIN_PWRGND21.5
- new net IO_101_12: PIN_AIN_PWRGND12.15, PIN_AIN_PWRGND21.3
- new net IO_101_13: PIN_AIN_PWRGND13.15, PIN_AIN_PWRGND21.1
- new net IO_101_14: PIN_AIN_PWRGND14.15, PIN_AIN_PWRGND21.14
- new net IO_101_15: PIN_AIN_PWRGND15.15, PIN_AIN_PWRGND21.12
- new net IO_101_16: PIN_AIN_PWRGND16.15, PIN_AIN_PWRGND21.10
- new net IO_101_17: PIN_AIN_PWRGND17.15, PIN_AIN_PWRGND21.8
- new net IO_101_18: PIN_AIN_PWRGND18.15, PIN_AIN_PWRGND21.6
- new net IO_101_19: PIN_AIN_PWRGND19.15, PIN_AIN_PWRGND21.4
- new net IO_101_2: PIN_AIN_PWRGND2.15, PIN_ANALOG_21.6
- new net IO_101_20: PIN_AIN_PWRGND20.15, PIN_AIN_PWRGND21.2
- new net IO_101_3: PIN_AIN_PWRGND3.15, PIN_ANALOG_21.8
- new net IO_101_4: PIN_AIN_PWRGND4.15, PIN_ANALOG_21.10
- new net IO_101_5: PIN_AIN_PWRGND5.15, PIN_ANALOG_21.12
- new net IO_101_6: PIN_AIN_PWRGND6.15, PIN_ANALOG_21.14
- new net IO_101_7: PIN_AIN_PWRGND21.13, PIN_AIN_PWRGND7.15
- new net IO_101_8: PIN_AIN_PWRGND21.11, PIN_AIN_PWRGND8.15
- new net IO_101_9: PIN_AIN_PWRGND21.9, PIN_AIN_PWRGND9.15
- new net IO_CLK_88_1: PIN_AIN_PWRGND1.5
- new net IO_CLK_88_2: PIN_AIN_PWRGND2.5
- new net IO_CLK_89_1: PIN_AIN_PWRGND1.7
- new net IO_CLK_89_2: PIN_AIN_PWRGND2.7
- new net IO_CLK_90_!: PIN_AIN_PWRGND1.9
- new net IO_CLK_90_2: PIN_AIN_PWRGND2.9
- new net IO_CLK_91_1: PIN_AIN_PWRGND1.11
- new net IO_CLK_91_2: PIN_AIN_PWRGND2.11
- new net L121_2: PIN_AIN_PWRGND2.4
- new net N$1: PIN_ANALOG_1.14, PIN_ANALOG_2.13
- new net N$10: PIN_ANALOG_2.8, PIN_ANALOG_3.7
- new net N$100: PIN_ANALOG_13.10, PIN_ANALOG_14.9
- new net N$101: PIN_ANALOG_13.12, PIN_ANALOG_14.11
- new net N$102: PIN_ANALOG_13.14, PIN_ANALOG_14.13
- new net N$104: PIN_ANALOG_14.2, PIN_ANALOG_15.1
- new net N$105: PIN_ANALOG_14.4, PIN_ANALOG_15.3
- new net N$106: PIN_ANALOG_14.6, PIN_ANALOG_15.5
- new net N$107: PIN_ANALOG_14.8, PIN_ANALOG_15.7
- new net N$108: PIN_ANALOG_14.10, PIN_ANALOG_15.9
- new net N$109: PIN_ANALOG_14.12, PIN_ANALOG_15.11
- new net N$11: PIN_ANALOG_2.10, PIN_ANALOG_3.9
- new net N$110: PIN_ANALOG_14.14, PIN_ANALOG_15.13
- new net N$112: PIN_ANALOG_15.2, PIN_ANALOG_16.1
- new net N$113: PIN_ANALOG_15.4, PIN_ANALOG_16.3
- new net N$114: PIN_ANALOG_15.6, PIN_ANALOG_16.5
- new net N$115: PIN_ANALOG_15.8, PIN_ANALOG_16.7
- new net N$116: PIN_ANALOG_15.10, PIN_ANALOG_16.9
- new net N$117: PIN_ANALOG_15.12, PIN_ANALOG_16.11
- new net N$118: PIN_ANALOG_15.14, PIN_ANALOG_16.13
- new net N$12: PIN_ANALOG_2.12, PIN_ANALOG_3.11
- new net N$120: PIN_ANALOG_16.2, PIN_ANALOG_17.1
- new net N$121: PIN_ANALOG_16.4, PIN_ANALOG_17.3
- new net N$122: PIN_ANALOG_16.6, PIN_ANALOG_17.5
- new net N$123: PIN_ANALOG_16.8, PIN_ANALOG_17.7
- new net N$124: PIN_ANALOG_16.10, PIN_ANALOG_17.9
- new net N$125: PIN_ANALOG_16.12, PIN_ANALOG_17.11
- new net N$126: PIN_ANALOG_16.14, PIN_ANALOG_17.13
- new net N$128: PIN_ANALOG_17.2, PIN_ANALOG_18.1
- new net N$129: PIN_ANALOG_17.4, PIN_ANALOG_18.3
- new net N$13: PIN_ANALOG_2.14, PIN_ANALOG_3.13
- new net N$130: PIN_ANALOG_17.6, PIN_ANALOG_18.5
- new net N$131: PIN_ANALOG_17.8, PIN_ANALOG_18.7
- new net N$132: PIN_ANALOG_17.10, PIN_ANALOG_18.9
- new net N$133: PIN_ANALOG_17.12, PIN_ANALOG_18.11
- new net N$134: PIN_ANALOG_17.14, PIN_ANALOG_18.13
- new net N$136: PIN_ANALOG_18.2, PIN_ANALOG_19.1
- new net N$137: PIN_ANALOG_18.4, PIN_ANALOG_19.3
- new net N$138: PIN_ANALOG_18.6, PIN_ANALOG_19.5
- new net N$139: PIN_ANALOG_18.8, PIN_ANALOG_19.7
- new net N$140: PIN_ANALOG_18.10, PIN_ANALOG_19.9
- new net N$141: PIN_ANALOG_18.12, PIN_ANALOG_19.11
- new net N$142: PIN_ANALOG_18.14, PIN_ANALOG_19.13
- new net N$144: PIN_ANALOG_19.2, PIN_ANALOG_20.1
- new net N$145: PIN_ANALOG_19.4, PIN_ANALOG_20.3
- new net N$146: PIN_ANALOG_19.6, PIN_ANALOG_20.5
- new net N$147: PIN_ANALOG_19.8, PIN_ANALOG_20.7
- new net N$148: PIN_ANALOG_19.10, PIN_ANALOG_20.9
- new net N$149: PIN_ANALOG_19.12, PIN_ANALOG_20.11
- new net N$15: PIN_ANALOG_3.2, PIN_ANALOG_4.1
- new net N$150: PIN_ANALOG_19.14, PIN_ANALOG_20.13
- new net N$152: PIN_ANALOG_20.2, PIN_ANALOG_21.1
- new net N$153: PIN_ANALOG_20.4, PIN_ANALOG_21.3
- new net N$154: PIN_ANALOG_20.6, PIN_ANALOG_21.5
- new net N$155: PIN_ANALOG_20.8, PIN_ANALOG_21.7
- new net N$156: PIN_ANALOG_20.10, PIN_ANALOG_21.9
- new net N$157: PIN_ANALOG_20.12, PIN_ANALOG_21.11
- new net N$158: PIN_ANALOG_20.14, PIN_ANALOG_21.13
- new net N$16: PIN_ANALOG_3.4, PIN_ANALOG_4.3
- new net N$19: PIN_ANALOG_3.8, PIN_ANALOG_4.7
- new net N$2: PIN_ANALOG_1.12, PIN_ANALOG_2.11
- new net N$20: PIN_ANALOG_3.10, PIN_ANALOG_4.9
- new net N$21: PIN_ANALOG_3.12, PIN_ANALOG_4.11
- new net N$22: PIN_ANALOG_3.14, PIN_ANALOG_4.13
- new net N$24: PIN_ANALOG_4.2, PIN_ANALOG_5.1
- new net N$25: PIN_ANALOG_4.4, PIN_ANALOG_5.3
- new net N$27: PIN_ANALOG_4.8, PIN_ANALOG_5.7
- new net N$28: PIN_ANALOG_4.10, PIN_ANALOG_5.9
- new net N$29: PIN_ANALOG_4.12, PIN_ANALOG_5.11
- new net N$3: PIN_ANALOG_1.10, PIN_ANALOG_2.9
- new net N$30: PIN_ANALOG_4.14, PIN_ANALOG_5.13
- new net N$32: PIN_ANALOG_5.2, PIN_ANALOG_6.1
- new net N$33: PIN_ANALOG_5.4, PIN_ANALOG_6.3
- new net N$35: PIN_ANALOG_5.8, PIN_ANALOG_6.7
- new net N$36: PIN_ANALOG_5.10, PIN_ANALOG_6.9
- new net N$37: PIN_ANALOG_5.12, PIN_ANALOG_6.11
- new net N$38: PIN_ANALOG_5.14, PIN_ANALOG_6.13
- new net N$4: PIN_ANALOG_1.8, PIN_ANALOG_2.7
- new net N$40: PIN_ANALOG_6.2, PIN_ANALOG_7.1
- new net N$41: PIN_ANALOG_6.4, PIN_ANALOG_7.3
- new net N$43: PIN_ANALOG_6.8, PIN_ANALOG_7.7
- new net N$44: PIN_ANALOG_6.10, PIN_ANALOG_7.9
- new net N$45: PIN_ANALOG_6.12, PIN_ANALOG_7.11
- new net N$46: PIN_ANALOG_6.14, PIN_ANALOG_7.13
- new net N$48: PIN_ANALOG_7.2, PIN_ANALOG_8.1
- new net N$49: PIN_ANALOG_7.4, PIN_ANALOG_8.3
- new net N$5: PIN_ANALOG_1.4, PIN_ANALOG_2.3
- new net N$51: PIN_ANALOG_7.8, PIN_ANALOG_8.7
- new net N$52: PIN_ANALOG_7.10, PIN_ANALOG_8.9
- new net N$53: PIN_ANALOG_7.12, PIN_ANALOG_8.11
- new net N$54: PIN_ANALOG_7.14, PIN_ANALOG_8.13
- new net N$56: PIN_ANALOG_8.2, PIN_ANALOG_9.1
- new net N$57: PIN_ANALOG_8.4, PIN_ANALOG_9.3
- new net N$59: PIN_ANALOG_8.8, PIN_ANALOG_9.7
- new net N$6: PIN_ANALOG_1.2, PIN_ANALOG_2.1
- new net N$60: PIN_ANALOG_8.10, PIN_ANALOG_9.9
- new net N$61: PIN_ANALOG_8.12, PIN_ANALOG_9.11
- new net N$62: PIN_ANALOG_8.14, PIN_ANALOG_9.13
- new net N$64: PIN_ANALOG_10.1, PIN_ANALOG_9.2
- new net N$65: PIN_ANALOG_10.3, PIN_ANALOG_9.4
- new net N$67: PIN_ANALOG_10.7, PIN_ANALOG_9.8
- new net N$68: PIN_ANALOG_10.9, PIN_ANALOG_9.10
- new net N$69: PIN_ANALOG_10.11, PIN_ANALOG_9.12
- new net N$7: PIN_ANALOG_2.2, PIN_ANALOG_3.1
- new net N$70: PIN_ANALOG_10.13, PIN_ANALOG_9.14
- new net N$72: PIN_ANALOG_10.2, PIN_ANALOG_11.1
- new net N$73: PIN_ANALOG_10.4, PIN_ANALOG_11.3
- new net N$74: PIN_ANALOG_10.6, PIN_ANALOG_11.5
- new net N$75: PIN_ANALOG_10.8, PIN_ANALOG_11.7
- new net N$76: PIN_ANALOG_10.10, PIN_ANALOG_11.9
- new net N$77: PIN_ANALOG_10.12, PIN_ANALOG_11.11
- new net N$78: PIN_ANALOG_10.14, PIN_ANALOG_11.13
- new net N$8: PIN_ANALOG_2.4, PIN_ANALOG_3.3
- new net N$80: PIN_ANALOG_11.2, PIN_ANALOG_12.1
- new net N$81: PIN_ANALOG_11.4, PIN_ANALOG_12.3
- new net N$82: PIN_ANALOG_11.6, PIN_ANALOG_12.5
- new net N$83: PIN_ANALOG_11.8, PIN_ANALOG_12.7
- new net N$84: PIN_ANALOG_11.10, PIN_ANALOG_12.9
- new net N$85: PIN_ANALOG_11.12, PIN_ANALOG_12.11
- new net N$86: PIN_ANALOG_11.14, PIN_ANALOG_12.13
- new net N$88: PIN_ANALOG_12.2, PIN_ANALOG_13.1
- new net N$89: PIN_ANALOG_12.4, PIN_ANALOG_13.3
- new net N$90: PIN_ANALOG_12.6, PIN_ANALOG_13.5
- new net N$91: PIN_ANALOG_12.8, PIN_ANALOG_13.7
- new net N$92: PIN_ANALOG_12.10, PIN_ANALOG_13.9
- new net N$93: PIN_ANALOG_12.12, PIN_ANALOG_13.11
- new net N$94: PIN_ANALOG_12.14, PIN_ANALOG_13.13
- new net N$96: PIN_ANALOG_13.2, PIN_ANALOG_14.1
- new net N$97: PIN_ANALOG_13.4, PIN_ANALOG_14.3
- new net N$98: PIN_ANALOG_13.6, PIN_ANALOG_14.5
- new net N$99: PIN_ANALOG_13.8, PIN_ANALOG_14.7
- net +5V: now also PIN_ANALOG_1.6, PIN_ANALOG_10.5, PIN_ANALOG_2.5, PIN_ANALOG_2.6, PIN_ANALOG_3.5, PIN_ANALOG_3.6, PIN_ANALOG_4.5, PIN_ANALOG_4.6, PIN_ANALOG_5.5, PIN_ANALOG_5.6, PIN_ANALOG_6.5, PIN_ANALOG_6.6, PIN_ANALOG_7.5, PIN_ANALOG_7.6, PIN_ANALOG_8.5, PIN_ANALOG_8.6, PIN_ANALOG_9.5, PIN_ANALOG_9.6; no longer PIN_ANALOG_IOEXP1.6
- net 5VINFROMRIGHT: now also PIN_ANALOG_1.5; no longer PIN_ANALOG_IOEXP1.5
- net AIN1: now also PIN_AIN_PWRGND1.2; no longer PIN_AIN_IO2_PWRGND.2
- net CLKINFROMRIGHT_26: now also PIN_ANALOG_1.1; no longer PIN_ANALOG_IOEXP1.1
- net GND: now also PIN_AIN_PWRGND1.1, PIN_AIN_PWRGND1.10, PIN_AIN_PWRGND1.12, PIN_AIN_PWRGND1.14, PIN_AIN_PWRGND1.16, PIN_AIN_PWRGND1.6, PIN_AIN_PWRGND1.8, PIN_AIN_PWRGND10.1, PIN_AIN_PWRGND10.10, PIN_AIN_PWRGND10.12, PIN_AIN_PWRGND10.14, PIN_AIN_PWRGND10.16, PIN_AIN_PWRGND10.6, PIN_AIN_PWRGND10.8, PIN_AIN_PWRGND11.1, PIN_AIN_PWRGND11.10, PIN_AIN_PWRGND11.12, PIN_AIN_PWRGND11.14, PIN_AIN_PWRGND11.16, PIN_AIN_PWRGND11.6, PIN_AIN_PWRGND11.8, PIN_AIN_PWRGND12.1, PIN_AIN_PWRGND12.10, PIN_AIN_PWRGND12.12, PIN_AIN_PWRGND12.14, PIN_AIN_PWRGND12.16, PIN_AIN_PWRGND12.6, PIN_AIN_PWRGND12.8, PIN_AIN_PWRGND13.1, PIN_AIN_PWRGND13.10, PIN_AIN_PWRGND13.12, PIN_AIN_PWRGND13.14, PIN_AIN_PWRGND13.16, PIN_AIN_PWRGND13.6, PIN_AIN_PWRGND13.8, PIN_AIN_PWRGND14.1, PIN_AIN_PWRGND14.10, PIN_AIN_PWRGND14.12, PIN_AIN_PWRGND14.14, PIN_AIN_PWRGND14.16, PIN_AIN_PWRGND14.6, PIN_AIN_PWRGND14.8, PIN_AIN_PWRGND15.1, PIN_AIN_PWRGND15.10, PIN_AIN_PWRGND15.12, PIN_AIN_PWRGND15.14, PIN_AIN_PWRGND15.16, PIN_AIN_PWRGND15.6, PIN_AIN_PWRGND15.8, PIN_AIN_PWRGND16.1, PIN_AIN_PWRGND16.10, PIN_AIN_PWRGND16.12, PIN_AIN_PWRGND16.14, PIN_AIN_PWRGND16.16, PIN_AIN_PWRGND16.6, PIN_AIN_PWRGND16.8, PIN_AIN_PWRGND17.1, PIN_AIN_PWRGND17.10, PIN_AIN_PWRGND17.12, PIN_AIN_PWRGND17.14, PIN_AIN_PWRGND17.16, PIN_AIN_PWRGND17.6, PIN_AIN_PWRGND17.8, PIN_AIN_PWRGND18.1, PIN_AIN_PWRGND18.10, PIN_AIN_PWRGND18.12, PIN_AIN_PWRGND18.14, PIN_AIN_PWRGND18.16, PIN_AIN_PWRGND18.6, PIN_AIN_PWRGND18.8, PIN_AIN_PWRGND19.1, PIN_AIN_PWRGND19.10, PIN_AIN_PWRGND19.12, PIN_AIN_PWRGND19.14, PIN_AIN_PWRGND19.16, PIN_AIN_PWRGND19.6, PIN_AIN_PWRGND19.8, PIN_AIN_PWRGND2.1, PIN_AIN_PWRGND2.10, PIN_AIN_PWRGND2.12, PIN_AIN_PWRGND2.14, PIN_AIN_PWRGND2.16, PIN_AIN_PWRGND2.6, PIN_AIN_PWRGND2.8, PIN_AIN_PWRGND20.1, PIN_AIN_PWRGND20.10, PIN_AIN_PWRGND20.12, PIN_AIN_PWRGND20.14, PIN_AIN_PWRGND20.16, PIN_AIN_PWRGND20.6, PIN_AIN_PWRGND20.8, PIN_AIN_PWRGND21.15, PIN_AIN_PWRGND21.16, PIN_AIN_PWRGND3.1, PIN_AIN_PWRGND3.10, PIN_AIN_PWRGND3.12, PIN_AIN_PWRGND3.14, PIN_AIN_PWRGND3.16, PIN_AIN_PWRGND3.6, PIN_AIN_PWRGND3.8, PIN_AIN_PWRGND4.1, PIN_AIN_PWRGND4.10, PIN_AIN_PWRGND4.12, PIN_AIN_PWRGND4.14, PIN_AIN_PWRGND4.16, PIN_AIN_PWRGND4.6, PIN_AIN_PWRGND4.8, PIN_AIN_PWRGND5.1, PIN_AIN_PWRGND5.10, PIN_AIN_PWRGND5.12, PIN_AIN_PWRGND5.14, PIN_AIN_PWRGND5.16, PIN_AIN_PWRGND5.6, PIN_AIN_PWRGND5.8, PIN_AIN_PWRGND6.1, PIN_AIN_PWRGND6.10, PIN_AIN_PWRGND6.12, PIN_AIN_PWRGND6.14, PIN_AIN_PWRGND6.16, PIN_AIN_PWRGND6.6, PIN_AIN_PWRGND6.8, PIN_AIN_PWRGND7.1, PIN_AIN_PWRGND7.10, PIN_AIN_PWRGND7.12, PIN_AIN_PWRGND7.14, PIN_AIN_PWRGND7.16, PIN_AIN_PWRGND7.6, PIN_AIN_PWRGND7.8, PIN_AIN_PWRGND8.1, PIN_AIN_PWRGND8.10, PIN_AIN_PWRGND8.12, PIN_AIN_PWRGND8.14, PIN_AIN_PWRGND8.16, PIN_AIN_PWRGND8.6, PIN_AIN_PWRGND8.8, PIN_AIN_PWRGND9.1, PIN_AIN_PWRGND9.10, PIN_AIN_PWRGND9.12, PIN_AIN_PWRGND9.14, PIN_AIN_PWRGND9.16, PIN_AIN_PWRGND9.6, PIN_AIN_PWRGND9.8, PIN_ANALOG_1.15, PIN_ANALOG_1.16, PIN_ANALOG_10.15, PIN_ANALOG_10.16, PIN_ANALOG_11.15, PIN_ANALOG_11.16, PIN_ANALOG_12.15, PIN_ANALOG_12.16, PIN_ANALOG_13.15, PIN_ANALOG_13.16, PIN_ANALOG_14.15, PIN_ANALOG_14.16, PIN_ANALOG_15.15, PIN_ANALOG_15.16, PIN_ANALOG_16.15, PIN_ANALOG_16.16, PIN_ANALOG_17.15, PIN_ANALOG_17.16, PIN_ANALOG_18.15, PIN_ANALOG_18.16, PIN_ANALOG_19.15, PIN_ANALOG_19.16, PIN_ANALOG_2.15, PIN_ANALOG_2.16, PIN_ANALOG_20.15, PIN_ANALOG_20.16, PIN_ANALOG_21.15, PIN_ANALOG_21.16, PIN_ANALOG_21.2, PIN_ANALOG_3.15, PIN_ANALOG_3.16, PIN_ANALOG_4.15, PIN_ANALOG_4.16, PIN_ANALOG_5.15, PIN_ANALOG_5.16, PIN_ANALOG_6.15, PIN_ANALOG_6.16, PIN_ANALOG_7.15, PIN_ANALOG_7.16, PIN_ANALOG_8.15, PIN_ANALOG_8.16, PIN_ANALOG_9.15, PIN_ANALOG_9.16; no longer PIN_AIN_IO2_PWRGND.1, PIN_AIN_IO2_PWRGND.10, PIN_AIN_IO2_PWRGND.12, PIN_AIN_IO2_PWRGND.14, PIN_AIN_IO2_PWRGND.16, PIN_AIN_IO2_PWRGND.6, PIN_AIN_IO2_PWRGND.8, PIN_ANALOG_IOEXP1.15, PIN_ANALOG_IOEXP1.16
- net L121: now also PIN_AIN_PWRGND1.4; no longer PIN_AIN_IO2_PWRGND.4
- net SERIALFROMRIGHT_TX_93: now also PIN_ANALOG_1.11; no longer PIN_ANALOG_IOEXP1.11
- net SERIALTORIGHT_RX_92: now also PIN_ANALOG_1.13; no longer PIN_ANALOG_IOEXP1.13
- net SPARERIGHT_99: now also PIN_ANALOG_1.3; no longer PIN_ANALOG_IOEXP1.3
- net TRIGINFROMRIGHT_86: now also PIN_ANALOG_1.9; no longer PIN_ANALOG_IOEXP1.9
- net TRIGOUTORIGHT_87: now also PIN_ANALOG_1.7; no longer PIN_ANALOG_IOEXP1.7
Other:
- note added: "Trrig board"
- note removed: "Back pinout 1"
- note removed: "Back pinout 2"

Commit message: ordered version of scope and backplane
Connections:
- removed net 5VINFROMRIGHT: PIN_ANALOG_1.5
- removed net N$106: PIN_ANALOG_14.6, PIN_ANALOG_15.5
- removed net N$114: PIN_ANALOG_15.6, PIN_ANALOG_16.5
- removed net N$122: PIN_ANALOG_16.6, PIN_ANALOG_17.5
- removed net N$130: PIN_ANALOG_17.6, PIN_ANALOG_18.5
- removed net N$138: PIN_ANALOG_18.6, PIN_ANALOG_19.5
- removed net N$146: PIN_ANALOG_19.6, PIN_ANALOG_20.5
- removed net N$154: PIN_ANALOG_20.6, PIN_ANALOG_21.5
- removed net N$74: PIN_ANALOG_10.6, PIN_ANALOG_11.5
- removed net N$82: PIN_ANALOG_11.6, PIN_ANALOG_12.5
- removed net N$90: PIN_ANALOG_12.6, PIN_ANALOG_13.5
- removed net N$98: PIN_ANALOG_13.6, PIN_ANALOG_14.5
- net +5V: now also PIN_ANALOG_1.5, PIN_ANALOG_10.6, PIN_ANALOG_11.5, PIN_ANALOG_11.6, PIN_ANALOG_12.5, PIN_ANALOG_12.6, PIN_ANALOG_13.5, PIN_ANALOG_13.6, PIN_ANALOG_14.5, PIN_ANALOG_14.6, PIN_ANALOG_15.5, PIN_ANALOG_15.6, PIN_ANALOG_16.5, PIN_ANALOG_16.6, PIN_ANALOG_17.5, PIN_ANALOG_17.6, PIN_ANALOG_18.5, PIN_ANALOG_18.6, PIN_ANALOG_19.5, PIN_ANALOG_19.6, PIN_ANALOG_20.5, PIN_ANALOG_20.6, PIN_ANALOG_21.5
- net IO_101_1: now also PIN_ANALOG_21.14; no longer PIN_ANALOG_21.4
- net IO_101_11: now also PIN_AIN_PWRGND21.9; no longer PIN_AIN_PWRGND21.5
- net IO_101_12: now also PIN_AIN_PWRGND21.11; no longer PIN_AIN_PWRGND21.3
- net IO_101_13: now also PIN_AIN_PWRGND21.13; no longer PIN_AIN_PWRGND21.1
- net IO_101_2: now also PIN_ANALOG_21.12; no longer PIN_ANALOG_21.6
- net IO_101_3: now also PIN_ANALOG_21.10; no longer PIN_ANALOG_21.8
- net IO_101_4: now also PIN_ANALOG_21.8; no longer PIN_ANALOG_21.10
- net IO_101_5: now also PIN_ANALOG_21.6; no longer PIN_ANALOG_21.12
- net IO_101_6: now also PIN_ANALOG_21.4; no longer PIN_ANALOG_21.14
- net IO_101_7: now also PIN_AIN_PWRGND21.1; no longer PIN_AIN_PWRGND21.13
- net IO_101_8: now also PIN_AIN_PWRGND21.3; no longer PIN_AIN_PWRGND21.11
- net IO_101_9: now also PIN_AIN_PWRGND21.5; no longer PIN_AIN_PWRGND21.9
Other:
- note added: "Trig board"
- note removed: "Trrig board"
