File: eagle/max10adc_v9.0_rack.brd (EAGLE design)
At the start: 98 x 100 mm, 193 parts, among them IC1 MAX19506, IC2 MAX19506, J1 MOLEX_BNC_73100-0105, J2 MOLEX_BNC_73100-0105, J3 MOLEX_BNC_73100-0105, J4 MOLEX_BNC_73100-0105, K1 AQY21SOP, K2 AQY21SOP, K3 AQY21SOP, K4 AQY21SOP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

Commit message: before routing
Parts:
- moved PIN_ANALOG_IOEXP1 10.2 mm to (-1.20, 43.4), flipped to the bottom
Other:
- board text added: "SPR R L"
- board text removed: "SPR L R"

Commit message: ordered version of scope and backplane
Routing:
- net +3V3: track 0.00 -> 428.4 mm, vias 0 -> 11
- net GND: track 0.00 -> 244.7 mm, vias 0 -> 100
- net L141_SCL: track 0.00 -> 194.8 mm, vias 0 -> 5
- net L21_SDA: track 0.00 -> 187.4 mm, vias 0 -> 6
- net +5V: track 0.00 -> 168.4 mm, vias 0 -> 1
- net VCCA: track 0.00 -> 167.9 mm, vias 0 -> 6
- net E_21_B0: track 0.00 -> 159.8 mm, vias 0 -> 2
- net A7: track 0.00 -> 159.1 mm, vias 0 -> 1
- net E_21_B4: track 0.00 -> 144.5 mm
- net A12: track 0.00 -> 129.6 mm, vias 0 -> 2
- net A6: track 0.00 -> 128.6 mm, vias 0 -> 1
- net N$11: track 0.00 -> 108.1 mm, vias 0 -> 3
- net A11: track 0.00 -> 105.4 mm, vias 0 -> 3
- net A14: track 0.00 -> 103.8 mm, vias 0 -> 1
- net A8: track 0.00 -> 102.6 mm, vias 0 -> 4
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
Commit message: add 6mm on top and bottom, to fit in sliders
Other:
- board size 98 x 100 mm -> 98 x 112 mm
Changed lines of the file:
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@@
 <drawing>
 <settings>
-<setting alwaysvectorfont="yes"/>
+<setting alwaysvectorfont="no"/>
 <setting keepoldvectorfont="yes"/>
 <setting verticaltext="up"/>
 </settings>
-<grid distance="0.1" unitdist="inch" unit="inch" style="dots" multiple="1" display="yes" altdistance="0.1" altunitdist="mm" altunit="mm"/>
+<grid distance="1" unitdist="mm" unit="mm" style="dots" multiple="1" display="yes" altdistance="0.1" altunitdist="mm" altunit="mm"/>
 <layers>
 <layer number="1" name="Top" color="4" fill="1" visible="yes" active="yes"/>
@@
 <hole x="-9.5" y="64.5" drill="1.6"/>
 <hole x="-9.5" y="-9.5" drill="1.6"/>
-<wire x1="-12" y1="-12" x2="-12" y2="88" width="0.1524" layer="20"/>
-<wire x1="-12" y1="88" x2="86" y2="88" width="0.1524" layer="20"/>
-<wire x1="86" y1="88" x2="86" y2="-12" width="0.1524" layer="20"/>
-<wire x1="86" y1="-12" x2="-12" y2="-12" width="0.1524" layer="20"/>
+<wire x1="-12" y1="-18" x2="-12" y2="94" width="0.1524" layer="20"/>
+<wire x1="-12" y1="94" x2="86" y2="94" width="0.1524" layer="20"/>
+<wire x1="86" y1="94" x2="86" y2="-18" width="0.1524" layer="20"/>
+<wire x1="86" y1="-18" x2="-12" y2="-18" width="0.1524" layer="20"/>
 <text x="39.7" y="63.6" size="0.8128" layer="21" font="vector" rot="R90">Right</text>
 <text x="39" y="59.6" size="0.8128" layer="21" font="vector" rot="R270">USB</text>
@@
 <element name="PIN_DISPLAY" library="Seeed-Connector" library_urn="urn:adsk.eagle:library:478" package="H10-2.54" package3d_urn="urn:adsk.eagle:package:33117/1" value="YELLOW-10P-2.54" x="2.1" y="58" smashed="yes" rot="R90">
 <attribute name="MPN" value="" x="2.1" y="58" size="1.778" layer="27" rot="R90" display="off"/>
+<attribute name="NAME" x="8.37" y="63.095" size="0.8128" layer="25" ratio="11" rot="R180"/>
 <attribute name="NAME" x="-0.44" y="58.635" size="1.27" layer="33" ratio="10" rot="R180"/>
-<attribute name="NAME" x="8.37" y="63.095" size="0.8128" layer="25" ratio="11" rot="R180"/>
 <attribute name="VALUE" x="3.37" y="60.54" size="0.889" layer="27" ratio="11" rot="R180"/>
 </element>
 <element name="PIN_IO_1" library="Seeed-Connector" library_urn="urn:adsk.eagle:library:478" package="H10-2.54" package3d_urn="urn:adsk.eagle:package:33117/1" value="YELLOW-10P-2.54" x="2.1" y="83.4" smashed="yes" rot="R270">
 <attribute name="MPN" value="" x="2.1" y="83.4" size="1.778" layer="27" rot="R270" display="off"/>
+<attribute name="NAME" x="1.83" y="80.305" size="0.8128" layer="25" ratio="11"/>
 <attribute name="NAME" x="4.64" y="82.765" size="1.27" layer="33" ratio="10"/>
-<attribute name="NAME" x="1.83" y="80.305" size="0.8128" layer="25" ratio="11"/>
 <attribute name="VALUE" x="0.83" y="80.86" size="0.889" layer="27" ratio="11"/>
 </element>

Commit message: put usb serial on bottom clean up wire stubs
Parts:
- moved C_OSC2 16.9 mm to (11.8, 78.5), turned to 180 degrees
- moved C_OSC1 9.51 mm to (-4.00, 78.5), turned to 0 degrees
- moved Y1 8.06 mm to (4.00, 77.2), flipped to the bottom, turned to 180 degrees
- moved U340G 5.39 mm to (1.70, 70.0), flipped to the bottom
- moved USB1 0.10 mm to (-10.4, 71.7), flipped to the bottom, turned to 90 degrees
Routing:
- net GND: track 244.7 -> 266.7 mm, vias 100 -> 99
- net SERIALFROMRIGHT_TX_93: track 78.7 -> 97.0 mm, vias 3 -> 2
- net IO_114: track 61.0 -> 72.9 mm
- net D7B: track 36.1 -> 24.5 mm
- net +3V3: track 428.4 -> 439.0 mm
- net CLKOUT_32: track 42.7 -> 34.8 mm
- net SERIALTORIGHT_RX_92: track 87.2 -> 80.1 mm, vias 1 -> 2
- net L21_SDA: track 187.4 -> 183.0 mm, vias 6 -> 5
- net IO_122: track 66.6 -> 70.9 mm, vias 1 -> 2
- net +5V: track 168.4 -> 172.6 mm
- net DPLUS: track 15.3 -> 11.8 mm
- net DMINUS: track 13.8 -> 17.0 mm
- net IO_118: track 65.5 -> 63.2 mm
- net N$31: track 7.48 -> 9.61 mm
- net 5VINFROMUSB: track 60.5 -> 59.6 mm
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