File: eagle/max10adc_v9.0_rack.sch (EAGLE design)
At the start: 193 parts, among them IC1 MAX19506, IC2 MAX19506, J1 MOLEX_BNC_73100-0105, J2 MOLEX_BNC_73100-0105, J3 MOLEX_BNC_73100-0105, J4 MOLEX_BNC_73100-0105, K1 AQY21SOP, K2 AQY21SOP, K3 AQY21SOP, K4 AQY21SOP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

Commit message: use max 4416EUA, which is available
Parts:
- removed U1, U2: MAX4416ESA, LMH6724:LMH6724MAX
- added IC3, IC4: MAX4416EUA+, SamacSys_Parts:MAX4416EUA+
Connections:
- net GND: now also IC3.VEE, IC4.VEE; no longer U1.V-, U2.V-
- net INA1: now also IC3.OUTA; no longer U1.OUTA
- net INA2: now also IC4.OUTA; no longer U2.OUTA
- net INAMINUS1: now also IC3.INA-; no longer U1.-INA
- net INAMINUS2: now also IC4.INA-; no longer U2.-INA
- net INB1: now also IC3.OUTB; no longer U1.OUTB
- net INB2: now also IC4.OUTB; no longer U2.OUTB
- net INBMINUS1: now also IC3.INB-; no longer U1.-INB
- net INBMINUS2: now also IC4.INB-; no longer U2.-INB
- net OFFSET1: now also IC3.INA+; no longer U1.+INA
- net OFFSET2: now also IC3.INB+; no longer U1.+INB
- net OFFSET3: now also IC4.INA+; no longer U2.+INA
- net OFFSET4: now also IC4.INB+; no longer U2.+INB
- net VCCA: now also IC3.VCC, IC4.VCC; no longer U1.V+, U2.V+
